File: PCA9685+L298/PCA9685+L298.kicad_pcb (KiCad board)
At the start: 2 copper layers, 62.2 x 25.4 mm, 40 parts, among them Q1 AOD417, U1 PCA9685

Commit message: .
Routing:
- net SCL: track 77.9 -> 75.2 mm
Changed lines of the file:
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@@
   )
   (setup
+    (stackup
+      (layer "F.SilkS" (type "Top Silk Screen"))
+      (layer "F.Paste" (type "Top Solder Paste"))
+      (layer "F.Mask" (type "Top Solder Mask") (thickness 0.01))
+      (layer "F.Cu" (type "copper") (thickness 0.035))
+      (layer "dielectric 1" (type "core") (thickness 1.51) (material "FR4") (epsilon_r 4.5) (loss_tangent 0.02))
+      (layer "B.Cu" (type "copper") (thickness 0.035))
+      (layer "B.Mask" (type "Bottom Solder Mask") (thickness 0.01))
+      (layer "B.Paste" (type "Bottom Solder Paste"))
+      (layer "B.SilkS" (type "Bottom Silk Screen"))
+      (copper_finish "None")
+      (dielectric_constraints no)
+    )
     (pad_to_mask_clearance 0)
     (pcbplotparams
@@
   (segment (start 149.7711 103.7336) (end 149.8121 103.7746) (width 0.254) (layer "B.Cu") (net 26))
   (segment (start 152.3521 101.0666) (end 177.7111 101.0666) (width 0.254) (layer "B.Cu") (net 26))
-  (segment (start 125.5141 99.5426) (end 122.8471 99.5426) (width 0.254) (layer "F.Cu") (net 27))
   (segment (start 169.3291 101.7016) (end 170.9801 101.7016) (width 0.254) (layer "F.Cu") (net 27))
-  (segment (start 133.5921 100.6086) (end 125.7681 100.6086) (width 0.254) (layer "F.Cu") (net 27))
-  (segment (start 122.8471 99.5426) (end 121.9581 100.4316) (width 0.254) (layer "F.Cu") (net 27))
+  (segment (start 133.7691 100.4316) (end 133.5921 100.6086) (width 0.254) (layer "F.Cu") (net 27))
   (segment (start 121.0691 103.6066) (end 119.2911 103.6066) (width 0.254) (layer "F.Cu") (net 27))
+  (segment (start 124.0671 100.6086) (end 121.0691 103.6066) (width 0.254) (layer "F.Cu") (net 27))
   (segment (start 168.8401 101.2126) (end 169.3291 101.7016) (width 0.254) (layer "F.Cu") (net 27))
-  (segment (start 125.7681 100.6086) (end 125.7681 99.7966) (width 0.254) (layer "F.Cu") (net 27))
-  (segment (start 125.7681 99.7966) (end 125.5141 99.5426) (width 0.254) (layer "F.Cu") (net 27))
+  (segment (start 133.5921 100.6086) (end 124.0671 100.6086) (width 0.254) (layer "F.Cu") (net 27))
   (segment (start 148.7551 102.7176) (end 149.6481 101.8246) (width 0.254) (layer "F.Cu") (net 27))
   (segment (start 149.6481 101.8246) (end 151.4189 101.8246) (width 0.254) (layer "F.Cu") (net 27))
-  (segment (start 121.9581 102.7176) (end 121.0691 103.6066) (width 0.254) (layer "F.Cu") (net 27))
   (segment (start 168.8401 100.3926) (end 168.8401 101.2126) (width 0.254) (layer "F.Cu") (net 27))
-  (segment (start 133.7691 100.4316) (end 133.5921 100.6086) (width 0.254) (layer "F.Cu") (net 27))
-  (segment (start 121.9581 100.4316) (end 121.9581 102.7176) (width 0.254) (layer "F.Cu") (net 27))
   (segment (start 170.9801 101.7016) (end 171.8691 102.5906) (width 0.254) (layer "F.Cu") (net 27))
   (segment (start 148.7551 105.0036) (end 148.7551 102.7176) (width 0.254) (layer "F.Cu") (net 27))

Commit message: 18.04.23
Parts:
- removed FID1, FID2: FIDUCIAL"", Adafruit PCA9685 rev C:FIDUCIAL_1MM
- removed JP1, JP2, JP5, JP6: , Adafruit PCA9685 rev C:3X04
- removed U$51: , Adafruit PCA9685 rev C:ADAFRUIT_5MM
- added C3: 1.0uF, Adafruit PCA9685 rev C:0805-NO, F.Cu at (83.6, 148.2)
- added C4: 1.0uF, Adafruit PCA9685 rev C:0805-NO, F.Cu at (83.6, 150.7)
- added C5: 1.0uF, Adafruit PCA9685 rev C:0805-NO, F.Cu at (83.6, 153.2)
- added C6: 10uF, Adafruit PCA9685 rev C:0805-NO, F.Cu at (76.5, 147.3)
- added C7: 10uF, Adafruit PCA9685 rev C:0805-NO, F.Cu at (76.5, 149.8)
- added C8: 1.0uF, Adafruit PCA9685 rev C:0805-NO, F.Cu at (76.5, 152.3)
- added C9: 1.0uF, Adafruit PCA9685 rev C:0805-NO, F.Cu at (76.5, 154.8)
- added D1: M7, Diode_SMD:D_SMA, F.Cu at (116.4, 164.3)
- added D10: M7, Diode_SMD:D_SMA, F.Cu at (144.9, 152.8)
- added D11: M7, Diode_SMD:D_SMA, F.Cu at (152.0, 152.8)
- added D12: M7, Diode_SMD:D_SMA, F.Cu at (144.9, 149.2)
- added D13: M7, Diode_SMD:D_SMA, F.Cu at (152.0, 149.2)
- added D14: M7, Diode_SMD:D_SMA, F.Cu at (144.9, 145.7)
- added D15: M7, Diode_SMD:D_SMA, F.Cu at (152.0, 145.7)
- added D16: M7, Diode_SMD:D_SMA, F.Cu at (144.9, 142.1)
- added D17: M7, Diode_SMD:D_SMA, F.Cu at (152.0, 142.1)
- added D18: M7, Diode_SMD:D_SMA, F.Cu at (164.0, 152.8)
- added D19: M7, Diode_SMD:D_SMA, F.Cu at (171.1, 152.8)
- added D2: M7, Diode_SMD:D_SMA, F.Cu at (125.8, 152.8)
- added D20: M7, Diode_SMD:D_SMA, F.Cu at (164.0, 149.2)
- added D21: M7, Diode_SMD:D_SMA, F.Cu at (171.1, 149.2)
- added D22: M7, Diode_SMD:D_SMA, F.Cu at (164.0, 145.7)
- added D23: M7, Diode_SMD:D_SMA, F.Cu at (171.1, 145.7)
- added D24: M7, Diode_SMD:D_SMA, F.Cu at (164.0, 142.1)
- added D25: M7, Diode_SMD:D_SMA, F.Cu at (171.1, 142.1)
- added D3: M7, Diode_SMD:D_SMA, F.Cu at (132.9, 152.8)
- added D4: M7, Diode_SMD:D_SMA, F.Cu at (125.8, 149.3)
- added D5: M7, Diode_SMD:D_SMA, F.Cu at (132.9, 149.3)
- added D6: M7, Diode_SMD:D_SMA, F.Cu at (125.8, 145.7)
- added D7: M7, Diode_SMD:D_SMA, F.Cu at (132.9, 145.7)
- added D8: M7, Diode_SMD:D_SMA, F.Cu at (125.8, 142.1)
- added D9: M7, Diode_SMD:D_SMA, F.Cu at (132.9, 142.1)
- added J10: TERMBLOCK_1X2, Adafruit PCA9685 rev C:TERMBLOCK_1X2-3.5MM, F.Cu at (171.3, 158.3)
- added J11: TERMBLOCK_1X2, Adafruit PCA9685 rev C:TERMBLOCK_1X2-3.5MM, F.Cu at (164.1, 158.3)
- added J12: QWIIC_RIGHT_ANGLE, Connectors:1X04_1MM_RA_STRESSRELIEF, F.Cu at (115.9, 103.9)
- added J2: QWIIC_RIGHT_ANGLE, Connectors:1X04_1MM_RA_STRESSRELIEF, F.Cu at (181.7, 104.7)
- added J3: Conn_01x04, Connector_PinHeader_2.54mm:PinHeader_1x04_P2.54mm_Vertical, F.Cu at (61.8, 148.7)
- added J4: TERMBLOCK_1X2, Adafruit PCA9685 rev C:TERMBLOCK_1X2-3.5MM, F.Cu at (133.1, 158.3)
- added J5: TERMBLOCK_1X2, Adafruit PCA9685 rev C:TERMBLOCK_1X2-3.5MM, F.Cu at (125.8, 158.3)
- added J6: Conn_01x04, Connector_PinHeader_2.54mm:PinHeader_1x04_P2.54mm_Vertical, F.Cu at (67.4, 148.4)
- added J7: TERMBLOCK_1X2, Adafruit PCA9685 rev C:TERMBLOCK_1X2-3.5MM, F.Cu at (152.2, 158.3)
- added J8: TERMBLOCK_1X2, Adafruit PCA9685 rev C:TERMBLOCK_1X2-3.5MM, F.Cu at (145.0, 158.3)
- added J9: Conn_01x04, Connector_PinHeader_2.54mm:PinHeader_1x04_P2.54mm_Vertical, F.Cu at (72.1, 148.4)
- added JP10: JUMPER-SMT_2_NC_TRACE_SILK, OLIMEX_Jumpers-FP:SJ_Closed, F.Cu at (91.1, 168.1)
- added JP11: JUMPER-SMT_2_NC_TRACE_SILK, OLIMEX_Jumpers-FP:SJ_Closed, B.Cu at (141.6, 136.0)
- added JP12: JUMPER-SMT_2_NC_TRACE_SILK, OLIMEX_Jumpers-FP:SJ_Closed, B.Cu at (141.6, 128.5)
- added JP13: JUMPER-SMT_2_NC_TRACE_SILK, OLIMEX_Jumpers-FP:SJ_Closed, B.Cu at (160.7, 136.0)
- added JP14: JUMPER-SMT_2_NC_TRACE_SILK, OLIMEX_Jumpers-FP:SJ_Closed, B.Cu at (160.7, 128.5)
- added JP7: JUMPER-SMT_2_NC_TRACE_SILK, OLIMEX_Jumpers-FP:SJ_Closed, B.Cu at (122.5, 136.0)
- added JP8: JUMPER-SMT_2_NC_TRACE_SILK, OLIMEX_Jumpers-FP:SJ_Closed, B.Cu at (122.5, 128.5)
- added JP9: JUMPER-SMT_2_NC_TRACE_SILK, OLIMEX_Jumpers-FP:SJ_Closed, B.Cu at (154.7, 94.7)
- added LED2: RED, Adafruit PCA9685 rev C:CHIPLED_0805_NOOUTLINE, F.Cu at (87.7, 168.6)
- added R5: 470, Adafruit PCA9685 rev C:_0805MP, F.Cu at (91.0, 170.9)
- added U2: L298HN, Silicon-Standard:POWERSO20_L298_PAD, F.Cu at (129.3, 132.2)
- added U3: L298HN, Silicon-Standard:POWERSO20_L298_PAD, F.Cu at (148.5, 132.2)
- added U4: L298HN, Silicon-Standard:POWERSO20_L298_PAD, F.Cu at (167.6, 132.2)
- added U5: ADS1115IDGS, Package_SO:TSSOP-10_3x3mm_P0.5mm, F.Cu at (92.7, 147.2)
- added U6: ADS1115IDGS, Package_SO:TSSOP-10_3x3mm_P0.5mm, F.Cu at (92.7, 151.8)
- added U7: ADS1115IDGS, Package_SO:TSSOP-10_3x3mm_P0.5mm, F.Cu at (92.7, 156.5)
- added U8: L7805, PCM_Package_TO_SOT_SMD_AKL:TO-252-3_TabPin2, F.Cu at (112.8, 119.5)
- C2: value (none) -> CPOL-USE3.5-8
- J1: value (none) -> TERMBLOCK_1X2
- JP3, JP4: value (none) -> PINHD-1X6CB
- SJ_A0, SJ_A1, SJ_A2, SJ_A3, SJ_A4, SJ_A5: value (none) -> SOLDERJUMPERREFLOW_NOPASTE
- TP1, TP2, TP3, TP4, TP5, TP6: value (none) -> TESTPOINTROUND1MM
- moved U$48 61.8 mm to (107.0, 174.9)
- moved U$50 61.7 mm to (174.6, 176.2)
- renumbered R7 to R3, R10 to R4
Connections:
- net A0 renamed /A0
- net A1 renamed /A1
- net A2 renamed /A2
- net A3 renamed /A3
- net A4 renamed /A4
- net A5 renamed /A5
- net OE renamed /OE
- net PWM0 renamed /PWM0
- net PWM1 renamed /PWM1
- net PWM10 renamed /PWM10
- net PWM11 renamed /PWM11
- net PWM12 renamed /PWM12
- net PWM13 renamed /PWM13
- net PWM14 renamed /PWM14
- net PWM15 renamed /PWM15
- net PWM2 renamed /PWM2
- net PWM3 renamed /PWM3
- net PWM4 renamed /PWM4
- net PWM5 renamed /PWM5
- net PWM6 renamed /PWM6
- net PWM7 renamed /PWM7
- net PWM8 renamed /PWM8
- net PWM9 renamed /PWM9
- net PWRIN renamed Net-(Q1-D)
- net SCL renamed /SCL
- net SDA renamed /SDA
- C1 pad 1: VCC -> 5.0V
- C2 pad +: 5.0V -> VCC
- LED1 pad A: VCC -> Net-(JP9-Pad1)
- Q1 pad 2: 5.0V -> VCC
- R11 pad 5: N$5 -> /P4
- R11 pad 6: N$4 -> /P5
- R11 pad 7: N$2 -> /P6
- R11 pad 8: N$3 -> /P7
- R13 pad 5: N$9 -> /P0
- R13 pad 6: N$8 -> /P1
- R13 pad 7: N$7 -> /P2
- R13 pad 8: N$6 -> /P3
- R14 pad 5: N$10 -> /P8
- R14 pad 6: N$11 -> /P9
- R14 pad 7: N$12 -> /P10
- R14 pad 8: N$13 -> /P11
- SJ_A0 pad 1: VCC -> 5.0V
- SJ_A1 pad 1: VCC -> 5.0V
- SJ_A2 pad 1: VCC -> 5.0V
- SJ_A3 pad 1: VCC -> 5.0V
- SJ_A4 pad 1: VCC -> 5.0V
- SJ_A5 pad 1: VCC -> 5.0V
- U1 pad 28: VCC -> 5.0V
Routing:
- net GND: track 33.0 -> 99.8 mm, vias 5 -> 8
- net VCC: track 92.7 -> 149.7 mm
- net Net-(D4-A): track 0.00 -> 55.4 mm
- net Net-(D12-A): track 0.00 -> 55.1 mm
- net Net-(D20-A): track 0.00 -> 54.9 mm
- net Net-(D2-A): track 0.00 -> 54.6 mm
- net Net-(D10-A): track 0.00 -> 53.9 mm
- net Net-(D18-A): track 0.00 -> 53.4 mm
- net Net-(D22-A): track 0.00 -> 38.1 mm
- net Net-(D6-A): track 0.00 -> 37.9 mm
- net Net-(D14-A): track 0.00 -> 36.6 mm
- net Net-(D24-A): track 0.00 -> 31.5 mm
- net Net-(D16-A): track 0.00 -> 30.1 mm
- net /P8: track 0.00 -> 29.2 mm
- net Net-(D8-A): track 0.00 -> 27.6 mm
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- removed copper zone on B.Cu, net GND
Other:
- board size 62.2 x 25.4 mm -> 97.2 x 101.7 mm

Commit message: 18.04.23
Parts:
- added J13: Conn_01x04, Connector_PinHeader_2.54mm:PinHeader_1x04_P2.54mm_Vertical, F.Cu at (76.0, 120.1)
- JP10: moved to B.Cu
- moved LED2 100.0 mm to (155.7, 95.3), turned to 90 degrees
- moved JP10 97.3 mm to (155.7, 95.3), turned to 180 degrees
- moved R5 97.0 mm to (152.9, 96.3), turned to -90 degrees
- moved U8 84.9 mm to (197.0, 130.4), turned to 180 degrees
- moved R4 18.2 mm to (151.3, 81.0)
- moved JP9 15.0 mm to (148.1, 81.3)
- moved LED1 15.0 mm to (148.1, 81.3)
- moved C1 13.7 mm to (114.5, 110.7)
- moved R3 12.7 mm to (135.1, 103.5)
- moved R12 10.8 mm to (159.7, 107.8)
- moved R2 10.3 mm to (158.4, 101.8)
- moved R13 9.15 mm to (137.9, 107.8)
- moved R1 7.41 mm to (154.4, 101.8)
- moved R14 7.18 mm to (155.7, 107.8)
- moved R11 6.83 mm to (141.9, 107.8)
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Connections:
- R2 pad 5: VCC -> 5.0V
- R2 pad 6: VCC -> 5.0V
Routing:
- net VCC: track 149.7 -> 110.8 mm
- net 5.0V: track 94.0 -> 117.3 mm, vias 3 -> 4
- net /SDA: track 94.0 -> 71.4 mm, vias 3 -> 4
- net GND: track 99.8 -> 78.1 mm, vias 8 -> 4
- net /A1: track 32.0 -> 44.6 mm
- net /PWM12: track 20.5 -> 8.55 mm
- net /A0: track 36.1 -> 48.0 mm
- net /PWM15: track 23.5 -> 11.6 mm
- net /PWM14: track 22.5 -> 10.8 mm
- net /PWM13: track 21.5 -> 9.81 mm
- net /P8: track 29.2 -> 17.8 mm
- net /A3: track 29.3 -> 40.1 mm
- net /PWM0: track 21.3 -> 10.7 mm
- net /P7: track 11.1 -> 0.51 mm
- net /PWM1: track 20.2 -> 9.76 mm
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Other:
- board size 97.2 x 101.7 mm -> 76.4 x 78.1 mm
- board text removed: "12"
- board text removed: "13"
- board text removed: "14"
- board text removed: "15"

Commit message: 18.04.23
Parts:
- removed J3, J6, J9: Conn_01x04, Connector_PinHeader_2.54mm:PinHeader_1x04_P2.54mm_Vertical
- removed U$54: , Adafruit PCA9685 rev C:PCBFEAT-REV-040
- added FID1: FIDUCIAL"", Adafruit PCA9685 rev C:FIDUCIAL_1MM, F.Cu at (70.9, 128.2)
- added FID2: FIDUCIAL"", Adafruit PCA9685 rev C:FIDUCIAL_1MM, F.Cu at (70.9, 131.2)
- added JP1: ~, Adafruit PCA9685 rev C:3X04, F.Cu at (121.6, 146.4)
- added JP2: ~, Adafruit PCA9685 rev C:3X04, F.Cu at (175.6, 146.4)
- added JP5: ~, Adafruit PCA9685 rev C:3X04, F.Cu at (84.5, 164.2)
- C2: value CPOL-USE3.5-8 -> 1000uF
- R4: value 470 -> 1k
- moved C4 103.1 mm to (178.2, 109.6)
- moved C8 100.0 mm to (165.9, 107.5), turned to 90 degrees
- moved U6 95.1 mm to (179.3, 112.3)
- moved J13 88.3 mm to (163.6, 109.0), turned to 180 degrees
- moved C9 74.2 mm to (133.8, 107.7), turned to 90 degrees
- moved C7 69.5 mm to (131.9, 107.7), turned to 90 degrees
- moved C6 68.6 mm to (128.3, 102.3), turned to 180 degrees
- moved D1 63.7 mm to (135.4, 103.5)
- moved C3 50.8 mm to (116.6, 109.5), turned to 180 degrees
- moved U5 42.8 mm to (117.7, 112.3)
- moved U8 37.0 mm to (170.5, 104.6), turned to 90 degrees
- moved C1 31.2 mm to (143.5, 99.2), turned to 90 degrees
- moved R4 23.0 mm to (132.7, 94.5), turned to 180 degrees
- moved JP9 14.4 mm to (142.6, 94.6), turned to 180 degrees
- moved LED1 14.4 mm to (142.6, 94.6), turned to 90 degrees
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Routing:
- net VCC: track 110.8 -> 388.0 mm, vias 0 -> 15
- net 3.3V: track 0.00 -> 180.4 mm, vias 0 -> 5
- net GND: track 78.1 -> 153.2 mm, vias 4 -> 23
- net 5.0V: track 117.3 -> 177.4 mm, vias 4 -> 8
- net Net-(U5-AIN3): track 0.00 -> 34.7 mm
- net Net-(U6-AIN0): track 0.00 -> 34.7 mm, vias 0 -> 1
- net Net-(U5-AIN1): track 0.00 -> 34.4 mm
- net Net-(U6-AIN1): track 0.00 -> 32.9 mm
- net Net-(U5-AIN0): track 0.00 -> 32.5 mm, vias 0 -> 1
- net Net-(U6-AIN2): track 0.00 -> 32.5 mm
- net Net-(U6-AIN3): track 0.00 -> 32.3 mm, vias 0 -> 1
- net Net-(U5-AIN2): track 0.00 -> 31.8 mm
- net /SCL: track 66.7 -> 88.5 mm, vias 3 -> 5
- net /SDA: track 71.4 -> 91.8 mm
- net /P0: track 15.2 -> 31.6 mm
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- added copper zone on B.Cu, net GND
- added copper zone on F.Cu, net GND
Other:
- board text removed: "+RW"
- board text removed: "0"
- board text removed: "1"
- board text removed: "10"
- board text removed: "11"
- board text removed: "2"
- board text removed: "3"
- board text removed: "4"
- board text removed: "5"
- board text removed: "6"
- board text removed: "7"
- board text removed: "8"
- board text removed: "9"

Commit message: rev 0
Parts:
- removed the C5 at (83.6, 153.2)
- removed FID1, FID2: FIDUCIAL"", Adafruit PCA9685 rev C:FIDUCIAL_1MM
- added C4: 1.0uF, Adafruit PCA9685 rev C:0805-NO, F.Cu at (116.5, 115.1)
- added JP2: ~, Adafruit PCA9685 rev C:3X02, F.Cu at (124.2, 145.2)
- JP5: footprint Adafruit PCA9685 rev C:3X04 -> Adafruit PCA9685 rev C:3X02
- moved JP5 90.3 mm to (172.7, 145.1)
- moved U6 45.9 mm to (117.7, 117.9)
- moved JP1 4.55 mm to (117.8, 143.9), turned to -90 degrees
- moved JP6 4.33 mm to (179.1, 143.9), turned to 90 degrees
- renumbered C4 to C5, JP2 to JP6, U7 to U6, U6 to U7
Connections:
- JP5 pad 3: Net-(U7-AIN0) (its old number) -> Net-(U6-AIN2)
- JP5 pad 6: Net-(U7-AIN1) (its old number) -> Net-(U6-AIN3)
- U6 pad 1: /SCL -> 3.3V
- U6 pad 10: /SDA -> /SCL
- U6 pad 4: Net-(U7-AIN0) (its old number) -> Net-(U6-AIN0)
- U6 pad 5: Net-(U7-AIN1) (its old number) -> Net-(U6-AIN1)
- U6 pad 6: Net-(U7-AIN2) (its old number) -> Net-(U6-AIN2)
- U6 pad 7: Net-(U7-AIN3) (its old number) -> Net-(U6-AIN3)
- U6 pad 9: /SCL -> /SDA
- U7 pad 1: 3.3V -> /SCL
- U7 pad 10: /SCL -> /SDA
- U7 pad 9: /SDA -> /SCL
Routing:
- net Net-(U6-AIN3): track 0.00 -> 78.4 mm, vias 0 -> 1
- net Net-(U6-AIN2): track 0.00 -> 73.5 mm, vias 0 -> 1
- net Net-(U6-AIN1): track 0.00 -> 36.9 mm
- net 3.3V: track 180.4 -> 214.4 mm, vias 5 -> 8
- net Net-(U6-AIN0): track 0.00 -> 32.3 mm
- net Net-(D18-A): track 58.0 -> 38.9 mm, vias 0 -> 2
- net GND: track 153.2 -> 167.4 mm, vias 23 -> 29
- net /SCL: track 88.5 -> 101.5 mm, vias 5 -> 7
- net Net-(D20-A): track 53.2 -> 40.4 mm, vias 0 -> 2
- net Net-(U5-AIN3): track 34.7 -> 41.8 mm, vias 0 -> 1
- net /SDA: track 91.8 -> 98.3 mm
- net Net-(U7-AIN0): track 34.7 -> 38.1 mm
- net Net-(U5-AIN2): track 31.8 -> 35.2 mm, vias 0 -> 1
- net Net-(U7-AIN3): track 32.3 -> 29.7 mm
- net Net-(U5-AIN1): track 34.4 -> 31.8 mm, vias 0 -> 1
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Other:
- board size 76.4 x 78.1 mm -> 69.2 x 57 mm

Commit message: 1
Parts:
- moved U$48 21.2 mm to (110.8, 158.4)
- moved U$50 20.5 mm to (184.9, 158.4)
Routing:
- net Net-(D8-A): track 33.5 -> 23.6 mm
- net Net-(D4-A): track 56.3 -> 49.6 mm, vias 0 -> 2
- net VCC: track 388.0 -> 392.3 mm
- net Net-(U6-AIN0): track 32.3 -> 28.8 mm
- net Net-(U6-AIN1): track 36.9 -> 33.3 mm
- net Net-(D2-A): track 56.9 -> 58.5 mm, vias 0 -> 2
- net 3.3V: track 214.4 -> 212.8 mm
- net GND: track 167.4 -> 166.6 mm
- net /SCL: track 101.5 -> 102.3 mm
- net /OE: track 57.2 -> 57.9 mm

Commit message: .
Parts:
- moved J13 0.12 mm to (163.6, 109.0)
- moved C3 0.11 mm to (116.5, 109.5)
- moved C4 0.11 mm to (116.4, 115.1)
- moved U5 0.11 mm to (117.6, 112.3)
- moved U6 0.11 mm to (117.6, 117.9)
- turned JP12 to 90 degrees
- turned JP14 to 90 degrees
- turned JP8 to 90 degrees
Connections:
- U2 pad PAD: (no net) -> GND
- U3 pad PAD: (no net) -> GND
- U4 pad PAD: (no net) -> GND
Routing:
- net GND: track 166.6 -> 419.3 mm, vias 29 -> 266
- net VCC: track 392.3 -> 418.0 mm, vias 15 -> 17
- net Net-(D2-A): track 58.5 -> 48.8 mm, vias 2 -> 5
- net 3.3V: track 212.8 -> 203.4 mm, vias 8 -> 7
- net Net-(D6-A): track 42.2 -> 36.6 mm
- net Net-(U5-AIN2): track 35.2 -> 40.2 mm
- net /P8: track 21.1 -> 25.6 mm, vias 0 -> 2
- net /P4: track 19.3 -> 23.1 mm, vias 0 -> 2
- net /P0: track 31.9 -> 34.5 mm
- net /SCL: track 102.3 -> 104.7 mm
- net /SDA: track 98.3 -> 100.8 mm, vias 4 -> 5
- net Net-(D10-A): track 54.8 -> 52.6 mm, vias 0 -> 2
- net Net-(U6-AIN2): track 73.5 -> 75.4 mm
- net Net-(U6-AIN3): track 78.4 -> 80.2 mm
- net Net-(U3-EnA): track 7.27 -> 9.02 mm
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
Commit message: 23.04.23
Parts:
- moved JP5 11.4 mm to (179.1, 135.6), turned to -90 degrees
- moved JP2 6.38 mm to (117.8, 145.8), turned to -90 degrees
- moved JP1 5.70 mm to (117.8, 138.2)
- moved JP6 0.61 mm to (179.1, 143.3), turned to -90 degrees
Connections:
- JP5 pad 1: GND -> Net-(U6-AIN2)
- JP5 pad 3: Net-(U6-AIN2) -> GND
- JP5 pad 4: GND -> Net-(U6-AIN3)
- JP5 pad 6: Net-(U6-AIN3) -> GND
- JP6 pad 1: GND -> Net-(U7-AIN0)
- JP6 pad 10: GND -> Net-(U7-AIN3)
- JP6 pad 12: Net-(U7-AIN3) -> GND
- JP6 pad 3: Net-(U7-AIN0) -> GND
- JP6 pad 4: GND -> Net-(U7-AIN1)
- JP6 pad 6: Net-(U7-AIN1) -> GND
- JP6 pad 7: GND -> Net-(U7-AIN2)
- JP6 pad 9: Net-(U7-AIN2) -> GND
- U2 pad : GND -> (no net)
- U2 pad PAD: GND -> (no net)
- U3 pad : GND -> (no net)
- U3 pad PAD: GND -> (no net)
- U4 pad : GND -> (no net)
- U4 pad PAD: GND -> (no net)
Routing:
- net GND: track 419.3 -> 716.7 mm
- net Net-(U7-AIN0): track 38.1 -> 1.98 mm
- net 3.3V: track 203.4 -> 173.7 mm
- net Net-(U6-AIN2): track 75.4 -> 85.4 mm
- net Net-(U5-AIN2): track 40.2 -> 31.4 mm
- net Net-(U7-AIN3): track 30.2 -> 37.2 mm
- net Net-(U6-AIN3): track 80.2 -> 86.9 mm
- net Net-(U7-AIN1): track 35.3 -> 29.5 mm
- net Net-(U5-AIN0): track 30.4 -> 24.7 mm
- net Net-(U5-AIN3): track 41.9 -> 36.2 mm
- net Net-(U5-AIN1): track 31.8 -> 26.1 mm
- net Net-(U6-AIN1): track 33.3 -> 30.2 mm
- net Net-(U7-AIN2): track 31.6 -> 33.8 mm
- net Net-(U6-AIN0): track 28.7 -> 30.6 mm
- net Net-(D2-A): track 48.8 -> 49.9 mm
Other:
- board size 69.2 x 57 mm -> 69.2 x 56.1 mm
