File: PCA9685+L298/PCA9685+L298.kicad_pcb (KiCad board)
At the start: 2 copper layers, 69.2 x 56.1 mm, 94 parts, among them J1 TERMBLOCK_1X2, J10 TERMBLOCK_1X2, J11 TERMBLOCK_1X2, J12 QWIIC_RIGHT_ANGLE, J13 Conn_01x04, J2 QWIIC_RIGHT_ANGLE, J4 TERMBLOCK_1X2, J5 TERMBLOCK_1X2, J7 TERMBLOCK_1X2, J8 TERMBLOCK_1X2, Q1 AOD417, U1 PCA9685, U2 L298HN, U3 L298HN, U4 L298HN, U5 ADS1115IDGS, U6 ADS1115IDGS, U7 ADS1115IDGS, U8 L7805

Commit message: .
Parts:
- moved U$48 13.9 mm to (116.6, 145.8)
- moved U$50 13.5 mm to (180.3, 145.8)
- moved JP1 7.21 mm to (117.8, 131.0)
- moved JP2 7.21 mm to (117.8, 138.6)
- moved JP5 6.00 mm to (179.1, 129.6)
- moved JP6 6.00 mm to (179.1, 137.3)
- moved U$47 3.97 mm to (116.6, 95.7)
- moved U$49 3.83 mm to (180.3, 95.7)
Connections:
- U2 pad : (no net) -> GND
- U2 pad PAD: (no net) -> GND
- U3 pad : (no net) -> GND
- U3 pad PAD: (no net) -> GND
- U4 pad : (no net) -> GND
- U4 pad PAD: (no net) -> GND
Routing:
- net 5.0V: track 176.9 -> 202.6 mm, vias 5 -> 11
- net Net-(U7-AIN0): track 1.98 -> 23.0 mm, vias 1 -> 0
- net Net-(U6-AIN2): track 85.4 -> 98.8 mm
- net 3.3V: track 173.7 -> 160.9 mm, vias 7 -> 6
- net VCC: track 418.0 -> 405.3 mm
- net GND: track 716.7 -> 728.2 mm, vias 266 -> 264
- net Net-(U5-AIN1): track 26.1 -> 18.8 mm
- net Net-(U6-AIN1): track 30.2 -> 23.0 mm
- net Net-(U5-AIN2): track 31.4 -> 24.2 mm
- net Net-(U6-AIN0): track 30.6 -> 23.4 mm
- net Net-(U5-AIN3): track 36.2 -> 29.0 mm
- net Net-(U5-AIN0): track 24.7 -> 17.5 mm
- net Net-(U7-AIN2): track 33.8 -> 27.6 mm, vias 0 -> 1
- net Net-(U7-AIN3): track 37.2 -> 31.7 mm, vias 1 -> 2
- net Net-(U7-AIN1): track 29.5 -> 24.7 mm
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Other:
- board size 69.2 x 56.1 mm -> 69.2 x 55.6 mm

Commit message: 28.04.23
Parts:
- removed the JP6 at (179.1, 137.3)
- added JP15: ~, Adafruit PCA9685 rev C:3X02, F.Cu at (200.4, 134.7)
- added JP16: ~, Adafruit PCA9685 rev C:3X02, F.Cu at (200.4, 139.8)
- added JP2: ~, Adafruit PCA9685 rev C:3X02, F.Cu at (96.6, 133.5)
- JP1: footprint Adafruit PCA9685 rev C:3X04 -> Adafruit PCA9685 rev C:3X02
- U2, U3, U4: footprint Silicon-Standard:POWERSO20_L298_PAD -> Package_TO_SOT_THT:TO-220-15_P2.54x2.54mm_StaggerOdd_Lead5.84mm_TabDown
- moved U4 111.0 mm to (81.2, 188.6), turned to 0 degrees
- moved U$48 26.4 mm to (90.2, 145.8)
- moved U$47 24.8 mm to (91.8, 95.7)
- moved U$49 24.1 mm to (204.3, 94.9)
- moved U$50 23.7 mm to (203.9, 145.7)
- moved U2 21.8 mm to (116.9, 136.8), turned to 0 degrees
- moved JP1 21.4 mm to (96.6, 128.4)
- moved C5 21.4 mm to (199.5, 109.6)
- moved JP4 21.4 mm to (196.6, 104.9)
- moved J2 21.4 mm to (198.8, 104.9)
- moved JP6 21.4 mm to (200.4, 129.6)
- moved U7 21.4 mm to (200.7, 112.3)
- moved J12 21.2 mm to (98.3, 104.9)
- moved U5 21.2 mm to (96.3, 112.3)
- moved U6 21.2 mm to (96.3, 117.9)
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- renumbered D16 to D10, D17 to D11, D14 to D12, D15 to D13, D12 to D14, D13 to D15, D10 to D16, D11 to D17, D24 to D18, D25 to D19, D8 to D2, D22 to D20, D23 to D21, D20 to D22, D21 to D23, D18 to D24, D19 to D25, D9 to D3, D6 to D4, D7 to D5, D4 to D6, D5 to D7, D2 to D8, D3 to D9, J11 to J10, J10 to J11, J5 to J4, J4 to J5, J8 to J7, J7 to J8, JP2 to JP5, JP5 to JP6
Connections:
- D10 pad 2: Net-(D16-A) -> Net-(D10-A)
- D11 pad 1: Net-(D16-A) -> Net-(D10-A)
- D12 pad 2: Net-(D14-A) -> Net-(D12-A)
- D13 pad 1: Net-(D14-A) -> Net-(D12-A)
- D14 pad 2: Net-(D12-A) -> Net-(D14-A)
- D15 pad 1: Net-(D12-A) -> Net-(D14-A)
- D16 pad 2: Net-(D10-A) -> Net-(D16-A)
- D17 pad 1: Net-(D10-A) -> Net-(D16-A)
- D18 pad 2: Net-(D24-A) -> Net-(D18-A)
- D19 pad 1: Net-(D24-A) -> Net-(D18-A)
- D2 pad 2: Net-(D8-A) -> Net-(D2-A)
- D20 pad 2: Net-(D22-A) -> Net-(D20-A)
- D21 pad 1: Net-(D22-A) -> Net-(D20-A)
- D22 pad 2: Net-(D20-A) -> Net-(D22-A)
- D23 pad 1: Net-(D20-A) -> Net-(D22-A)
- D24 pad 2: Net-(D18-A) -> Net-(D24-A)
- D25 pad 1: Net-(D18-A) -> Net-(D24-A)
- D3 pad 1: Net-(D8-A) -> Net-(D2-A)
- D4 pad 2: Net-(D6-A) -> Net-(D4-A)
- D5 pad 1: Net-(D6-A) -> Net-(D4-A)
- D6 pad 2: Net-(D4-A) -> Net-(D6-A)
- D7 pad 1: Net-(D4-A) -> Net-(D6-A)
- D8 pad 2: Net-(D2-A) -> Net-(D8-A)
- D9 pad 1: Net-(D2-A) -> Net-(D8-A)
- J10 pad 1: Net-(D22-A) -> Net-(D20-A)
- J10 pad 2: Net-(D24-A) -> Net-(D18-A)
- J11 pad 1: Net-(D18-A) -> Net-(D24-A)
- J11 pad 2: Net-(D20-A) -> Net-(D22-A)
- J4 pad 1: Net-(D6-A) -> Net-(D4-A)
- J4 pad 2: Net-(D8-A) -> Net-(D2-A)
- J5 pad 1: Net-(D2-A) -> Net-(D8-A)
- J5 pad 2: Net-(D4-A) -> Net-(D6-A)
- J7 pad 1: Net-(D14-A) -> Net-(D12-A)
- J7 pad 2: Net-(D16-A) -> Net-(D10-A)
- J8 pad 1: Net-(D10-A) -> Net-(D16-A)
- J8 pad 2: Net-(D12-A) -> Net-(D14-A)
- U2 pad : GND -> (no net)
- U2 pad 10: /P1 -> /P2
- U2 pad 12: /P0 -> /P3
- U2 pad 5: /P3 -> /P0
- U2 pad 7: /P2 -> /P1
- U3 pad : GND -> (no net)
- U3 pad 10: /P5 -> /P6
- U3 pad 12: /P4 -> /P7
- U3 pad 5: /P7 -> /P4
- U3 pad 7: /P6 -> /P5
- U4 pad : GND -> (no net)
- U4 pad 10: /P9 -> /P10
- U4 pad 12: /P8 -> /P11
- U4 pad 5: /P11 -> /P8
- U4 pad 7: /P10 -> /P9
Routing:
- net GND: track 728.2 -> 666.9 mm, vias 264 -> 68
- net Net-(D8-A): track 23.6 -> 83.9 mm, vias 0 -> 6
- net Net-(D6-A): track 36.6 -> 80.4 mm, vias 0 -> 6
- net Net-(D14-A): track 36.6 -> 76.1 mm, vias 0 -> 6
- net Net-(D16-A): track 30.1 -> 68.7 mm, vias 0 -> 6
- net 5.0V: track 202.6 -> 173.2 mm, vias 11 -> 2
- net Net-(D24-A): track 32.1 -> 58.1 mm, vias 0 -> 6
- net /P5: track 4.00 -> 28.8 mm
- net Net-(D12-A): track 54.3 -> 31.5 mm, vias 2 -> 0
- net Net-(D22-A): track 38.2 -> 60.6 mm, vias 0 -> 6
- net /P7: track 8.11 -> 29.3 mm
- net /P6: track 6.19 -> 27.3 mm
- net /P8: track 25.6 -> 5.59 mm, vias 2 -> 0
- net Net-(U6-AIN2): track 98.8 -> 78.9 mm
- net Net-(D20-A): track 40.6 -> 24.2 mm, vias 2 -> 0
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Other:
- board size 69.2 x 55.6 mm -> 120.4 x 81.1 mm
