File: Rev0/Rev0.kicad_pcb (KiCad board)
At the start: 2 copper layers, 69.2 x 55.6 mm, 96 parts, among them J1 TERMBLOCK_1X2, J10 TERMBLOCK_1X2, J11 TERMBLOCK_1X2, J12 QWIIC_RIGHT_ANGLE, J13 Conn_01x04, J2 QWIIC_RIGHT_ANGLE, J4 TERMBLOCK_1X2, J5 TERMBLOCK_1X2, J7 TERMBLOCK_1X2, J8 TERMBLOCK_1X2, Q1 AOD417, U1 PCA9685, U2 L298P, U3 L298P, U4 L298P, U5 ADS1115IDGS, U6 ADS1115IDGS, U7 ADS1115IDGS, U8 L7805

Commit message: .
Parts:
- removed the C5 at (178.2, 109.6)
- removed D10, D11, D12, D13, D14, D15, D16, D17, D18, D19, D20, D21, D22, D23, D24, D25, D4, D5, D6, D7, D8, D9: M7, Diode_SMD:D_SMA
- removed the D3 at (132.9, 139.5)
- removed JP10: JUMPER-SMT_2_NC_TRACE_SILK, OLIMEX_Jumpers-FP:SJ_Closed
- removed JP16, JP6: ~, Adafruit PCA9685 rev C:3X02
- removed the JP5 at (117.8, 139.8)
- removed LED2: RED, Adafruit PCA9685 rev C:CHIPLED_0805_NOOUTLINE
- added C10: 0.1uF, Capacitor_SMD:C_0603_1608Metric, F.Cu at (158.3, 86.4)
- added C11: 0.1uF, Capacitor_SMD:C_0603_1608Metric, F.Cu at (166.8, 114.6)
- added C13: 47uF/35v, Capacitor_THT:C_Radial_D6.3mm_H11.0mm_P2.50mm, F.Cu at (163.1, 87.8)
- added C14: 47uF/35v, Capacitor_THT:C_Radial_D6.3mm_H11.0mm_P2.50mm, F.Cu at (163.1, 102.2)
- added C15: 47uF/35v, Capacitor_THT:C_Radial_D6.3mm_H11.0mm_P2.50mm, F.Cu at (163.1, 116.7)
- added C16: 0.1uF, Capacitor_SMD:C_0603_1608Metric, F.Cu at (165.8, 58.5)
- added C17: 0.1uF, Capacitor_SMD:C_0603_1608Metric, F.Cu at (151.8, 62.1)
- added C18: 0.1uF, Capacitor_SMD:C_0603_1608Metric, F.Cu at (139.6, 114.0)
- added C6: 0.1uF, Capacitor_SMD:C_0603_1608Metric, F.Cu at (158.3, 115.2)
- added C7: 0.1uF, Capacitor_SMD:C_0603_1608Metric, F.Cu at (166.8, 85.8)
- added G***: LOGO, Graphics:Hasatio_logo_micro, F.Cu at (133.5, 65.7)
- added G***: LOGO, Graphics:Hasatio_logo_mini, B.Cu at (145.6, 102.9)
- added G***: LOGO, Graphics:qr-WaterQualityControl, B.Cu at (122.8, 124.6)
- added J10: TERMBLOCK_1X2, Adafruit PCA9685 rev C:TERMBLOCK_1X2-3.5MM, F.Cu at (142.2, 124.8)
- added J11: TERMBLOCK_1X2, Adafruit PCA9685 rev C:TERMBLOCK_1X2-3.5MM, F.Cu at (149.4, 124.8)
- added J12: TERMBLOCK_1X2, Adafruit PCA9685 rev C:TERMBLOCK_1X2-3.5MM, F.Cu at (156.6, 124.8)
- added J19: TERMBLOCK_1X2, Adafruit PCA9685 rev C:TERMBLOCK_1X2-3.5MM, F.Cu at (115.6, 67.7)
- added J20: TERMBLOCK_1X2, Adafruit PCA9685 rev C:TERMBLOCK_1X2-3.5MM, F.Cu at (115.6, 74.9)
- added J21: TERMBLOCK_1X2, Adafruit PCA9685 rev C:TERMBLOCK_1X2-3.5MM, F.Cu at (115.6, 82.1)
- added J22: TERMBLOCK_1X2, Adafruit PCA9685 rev C:TERMBLOCK_1X2-3.5MM, F.Cu at (115.6, 89.3)
- added J23: TERMBLOCK_1X2, Adafruit PCA9685 rev C:TERMBLOCK_1X2-3.5MM, F.Cu at (115.6, 96.6)
- added J24: TERMBLOCK_1X2, Adafruit PCA9685 rev C:TERMBLOCK_1X2-3.5MM, F.Cu at (115.6, 103.8)
- added J25: TERMBLOCK_1X2, Adafruit PCA9685 rev C:TERMBLOCK_1X2-3.5MM, F.Cu at (115.6, 111.0)
- added J26: TERMBLOCK_1X2, Adafruit PCA9685 rev C:TERMBLOCK_1X2-3.5MM, F.Cu at (115.6, 118.2)
- added J28: Conn_01x02, Connector_PinHeader_2.54mm:PinHeader_1x02_P2.54mm_Vertical, F.Cu at (120.9, 69.0)
- added J29: Conn_01x02, Connector_PinHeader_2.54mm:PinHeader_1x02_P2.54mm_Vertical, F.Cu at (120.9, 76.2)
- added J30: Conn_01x02, Connector_PinHeader_2.54mm:PinHeader_1x02_P2.54mm_Vertical, F.Cu at (120.9, 83.4)
- added J31: Conn_01x02, Connector_PinHeader_2.54mm:PinHeader_1x02_P2.54mm_Vertical, F.Cu at (120.9, 90.6)
- added J32: Conn_01x02, Connector_PinHeader_2.54mm:PinHeader_1x02_P2.54mm_Vertical, F.Cu at (120.9, 97.8)
- added J33: Conn_01x02, Connector_PinHeader_2.54mm:PinHeader_1x02_P2.54mm_Vertical, F.Cu at (120.9, 105.0)
- added J34: Conn_01x02, Connector_PinHeader_2.54mm:PinHeader_1x02_P2.54mm_Vertical, F.Cu at (120.9, 112.2)
- added J35: Conn_01x02, Connector_PinHeader_2.54mm:PinHeader_1x02_P2.54mm_Vertical, F.Cu at (120.9, 119.5)
- added JP9: JUMPER-SMT_2_NC_TRACE_SILK, OLIMEX_Jumpers-FP:SJ_Closed, B.Cu at (158.0, 115.2)
- added R10: 10K, Resistor_SMD:R_0603_1608Metric, F.Cu at (123.5, 74.4)
- added R15: 10K, Resistor_SMD:R_0603_1608Metric, F.Cu at (142.6, 114.0)
- added R16: 750, Resistor_SMD:R_0603_1608Metric, F.Cu at (123.5, 77.4)
- added R17: 10K, Resistor_SMD:R_0603_1608Metric, F.Cu at (123.5, 80.4)
- added R18: 750, Resistor_SMD:R_0603_1608Metric, F.Cu at (123.5, 83.4)
- added R19: 10K, Resistor_SMD:R_0603_1608Metric, F.Cu at (123.5, 86.4)
- added R20: 750, Resistor_SMD:R_0603_1608Metric, F.Cu at (123.5, 89.5)
- added R21: 750, Resistor_SMD:R_0603_1608Metric, F.Cu at (123.5, 92.5)
- added R22: 100, Resistor_SMD:R_0603_1608Metric, F.Cu at (123.5, 95.5)
- added R23: 750, Resistor_SMD:R_0603_1608Metric, F.Cu at (123.5, 98.5)
- added R24: 100, Resistor_SMD:R_0603_1608Metric, F.Cu at (123.5, 101.5)
- added R25: 750, Resistor_SMD:R_0603_1608Metric, F.Cu at (123.5, 104.5)
- added R26: 100, Resistor_SMD:R_0603_1608Metric, F.Cu at (123.5, 107.5)
- added R27: 750, Resistor_SMD:R_0603_1608Metric, F.Cu at (123.5, 110.5)
- added R28: 100, Resistor_SMD:R_0603_1608Metric, F.Cu at (123.5, 113.5)
- added R30: 1.5k, Adafruit PCA9685 rev C:RESPACK_4X0603, F.Cu at (157.7, 118.1)
- added R31: 100k, Resistor_SMD:R_0603_1608Metric, F.Cu at (156.3, 72.2)
- added R32: 10K, Resistor_SMD:R_0603_1608Metric, F.Cu at (151.8, 59.1)
- added R33: 10K, Resistor_SMD:R_0603_1608Metric, F.Cu at (148.5, 114.0)
- added R34: 10K, Resistor_SMD:R_0603_1608Metric, F.Cu at (145.5, 114.0)
- added R4: 1k, Resistor_SMD:R_0603_1608Metric, F.Cu at (122.1, 51.8)
- added R6: 250m/1w, Resistor_SMD:R_1206_3216Metric, F.Cu at (166.4, 95.2)
- added R7: 250m/1w, Resistor_SMD:R_1206_3216Metric, F.Cu at (166.4, 109.6)
- added R8: 10K, Resistor_SMD:R_0603_1608Metric, F.Cu at (123.5, 68.4)
- added R9: 750, Resistor_SMD:R_0603_1608Metric, F.Cu at (123.5, 71.4)
- added REF**: Converter_DCDC_RECOM_R-78B-2.0_THT, Converter_DCDC:Converter_DCDC_RECOM_R-78B-2.0_THT, F.Cu at (151.3, 77.7)
- added Sign_Pb-Free: , OLIMEX_LOGOs-FP:LOGO_PBFREE, B.Cu at (156.5, 66.2)
- added Sign_RoHS: Val**, OLIMEX_LOGOs-FP:LOGO_ROHS_1, B.Cu at (173.6, 77.9)
- added U10: PC817, Package_DIP:DIP-4_W7.62mm_SMDSocket_SmallPads, F.Cu at (129.7, 83.0)
- added U11: PC817, Package_DIP:DIP-4_W7.62mm_SMDSocket_SmallPads, F.Cu at (129.7, 88.8)
- added U12: PC817, Package_DIP:DIP-4_W7.62mm_SMDSocket_SmallPads, F.Cu at (129.7, 94.5)
- added U13: PC817, Package_DIP:DIP-4_W7.62mm_SMDSocket_SmallPads, F.Cu at (129.7, 100.3)
- added U14: PC817, Package_DIP:DIP-4_W7.62mm_SMDSocket_SmallPads, F.Cu at (129.7, 106.0)
- added U15: PC817, Package_DIP:DIP-4_W7.62mm_SMDSocket_SmallPads, F.Cu at (129.7, 111.8)
- added U16: ADS1115IDGS, Package_SO:TSSOP-10_3x3mm_P0.5mm, F.Cu at (135.0, 118.9)
- added U17: ADS1115IDGS, Package_SO:TSSOP-10_3x3mm_P0.5mm, F.Cu at (151.2, 119.5)
- added U9: PC817, Package_DIP:DIP-4_W7.62mm_SMDSocket_SmallPads, F.Cu at (129.7, 77.2)
- C1: footprint Adafruit PCA9685 rev C:0805-NO -> Capacitor_SMD:C_0603_1608Metric
- C12: renamed from C7; footprint Adafruit PCA9685 rev C:0805-NO -> Capacitor_SMD:C_0603_1608Metric
- C2: value 1000uF -> 1000uF/35v; footprint Adafruit PCA9685 rev C:E3,5-8 -> Capacitor_THT:C_Radial_D10.0mm_H20.0mm_P5.00mm
- C3, C4, C8, C9: value 1.0uF -> 0.1uF; footprint Adafruit PCA9685 rev C:0805-NO -> Capacitor_SMD:C_0603_1608Metric
- C5: renamed from C6; value 10uF -> 10uF/35v; footprint Adafruit PCA9685 rev C:0805-NO -> Capacitor_SMD:C_0603_1608Metric
- D1: value M7 -> GREEN; footprint Diode_SMD:D_SMA -> LED_SMD:LED_0603_1608Metric
- D2: value M7 -> Z1SMA4740
- D3: renamed from LED1; value GREEN -> RED; footprint Adafruit PCA9685 rev C:CHIPLED_0805_NOOUTLINE -> LED_SMD:LED_0603_1608Metric
- J13: value Conn_01x04 -> TERMBLOCK_1X2; footprint Connector_PinHeader_2.54mm:PinHeader_1x04_P2.54mm_Vertical -> Adafruit PCA9685 rev C:TERMBLOCK_1X2-3.5MM
- JP1: renamed from JP2; value ~ -> Conn_02x03
- JP12, JP13, JP14: value JUMPER-SMT_2_NC_TRACE_SILK -> Conn_02x03; footprint OLIMEX_Jumpers-FP:SJ_Closed -> Adafruit PCA9685 rev C:3X02; moved to F.Cu
- JP15: value ~ -> Conn_02x03
- JP2: renamed from JP1; value ~ -> Conn_02x03
- R1, R2: value 10K -> 10k
- R29: renamed from R4; footprint Adafruit PCA9685 rev C:_0805MP -> Resistor_SMD:R_0603_1608Metric
- R3: footprint Adafruit PCA9685 rev C:0805-NO -> Resistor_SMD:R_0603_1608Metric
- R5: value 470 -> 250m/1w; footprint Adafruit PCA9685 rev C:_0805MP -> Resistor_SMD:R_1206_3216Metric
- U2, U3, U4: value L298P -> DRV8870DDA; footprint Silicon-Standard:POWERSO20_L298_PAD -> Package_SO:Texas_HTSOP-8-1EP_3.9x4.9mm_P1.27mm_EP2.95x4.9mm_Mask2.4x3.1mm_ThermalVias
- U5: value ADS1115IDGS -> K7805-2000R3L; footprint Package_SO:TSSOP-10_3x3mm_P0.5mm -> Converter_DCDC:Converter_DCDC_RECOM_R-78HB-0.5L_THT
- U6: value ADS1115IDGS -> TCA9406DC; footprint Package_SO:TSSOP-10_3x3mm_P0.5mm -> PCM_Package_SO_AKL:SSOP-8_2.95x2.8mm_P0.65mm
- U7: value ADS1115IDGS -> MCP23008-xSO; footprint Package_SO:TSSOP-10_3x3mm_P0.5mm -> Package_SO:SOIC-18W_7.5x11.6mm_P1.27mm
- U8: value L7805 -> PC817; footprint PCM_Package_TO_SOT_SMD_AKL:TO-252-3_TabPin2 -> Package_DIP:DIP-4_W7.62mm_SMDSocket_SmallPads
- moved JP15 83.6 mm to (160.5, 53.2), turned to 0 degrees
- moved U6 73.2 mm to (162.2, 59.8), turned to 180 degrees
- moved JP13 70.2 mm to (150.3, 53.2), turned to 0 degrees
- moved D2 70.1 mm to (156.6, 76.5), turned to 90 degrees
- moved JP11 68.9 mm to (122.0, 56.5), turned to 180 degrees
- moved J4 63.0 mm to (171.1, 81.9), turned to 90 degrees
- moved JP14 62.1 mm to (155.4, 53.2), turned to 0 degrees
- moved JP12 62.0 mm to (145.3, 53.2), turned to 0 degrees
- moved J5 56.9 mm to (171.1, 89.2), turned to 90 degrees
- moved SJ_A1 54.0 mm to (139.0, 52.1)
- moved SJ_A2 54.0 mm to (136.5, 52.1)
- moved SJ_A4 54.0 mm to (131.4, 52.1)
- moved SJ_A5 54.0 mm to (128.8, 52.1)
- moved SJ_A0 54.0 mm to (141.5, 52.1)
- moved SJ_A3 54.0 mm to (133.9, 52.1)
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- renumbered J12 to J2, J2 to J3, J10 to J4, J11 to J5, J7 to J6, J8 to J7, J4 to J8, J5 to J9, JP9 to JP5
Connections:
- C1 pad 1: 5.0V -> +5V
- C12 pad 1: 5.0V -> +5V
- C3 pad 1: 3.3V -> +5V
- C4 pad 1: 3.3V -> +5V
- C8 pad 1: VCC -> +5V
- C9 pad 1: 5.0V -> VCC
- D1 pad 1: VCC -> Net-(D1-K)
- D1 pad 2: 5.0V -> Net-(D1-A)
- J1 pad 1: Net-(Q1-D) -> GND
- J1 pad 2: GND -> Net-(Q1-D)
- J13 pad 1: Net-(J13-Pin_1) -> /Ain7
- J13 pad 2: Net-(J13-Pin_2) -> GND
- J2 pad 2: 3.3V -> +3.3V
- J2 pad 3: /SDA -> /SDA_A
- J2 pad 4: /SCL -> /SCL_A
- J3 pad 2: 3.3V -> +3.3V
- J3 pad 3: /SDA -> /SDA_A
- J3 pad 4: /SCL -> /SCL_A
- J4 pad 1: Net-(D20-A) -> Net-(U2-OUT2)
- J4 pad 2: Net-(D18-A) -> GND
- J5 pad 1: Net-(D24-A) -> Net-(U2-OUT1)
- J5 pad 2: Net-(D22-A) -> GND
- J6 pad 1: Net-(D12-A) -> Net-(U3-OUT2)
- J6 pad 2: Net-(D10-A) -> GND
- J7 pad 1: Net-(D16-A) -> Net-(U3-OUT1)
- J7 pad 2: Net-(D14-A) -> GND
- J8 pad 1: Net-(D4-A) -> Net-(U4-OUT2)
- J8 pad 2: Net-(D2-A) -> GND
- J9 pad 1: Net-(D8-A) -> Net-(U4-OUT1)
- J9 pad 2: Net-(D6-A) -> GND
- JP1 pad 2: 3.3V -> +5V
- JP1 pad 3: Net-(U5-AIN2) -> /Ain2
- JP1 pad 5: 3.3V -> +5V
- JP1 pad 6: Net-(U5-AIN3) -> /Ain3
- JP11 pad 1: Net-(U3-EnB) -> Net-(D1-A)
- JP11 pad 2: 5.0V -> +5V
- JP12 pad 1: Net-(U3-EnA) -> /P8
- JP12 pad 2: 5.0V -> +5V
- JP13 pad 1: Net-(U4-EnB) -> /P10
- JP13 pad 2: 5.0V -> +5V
- JP14 pad 1: Net-(U4-EnA) -> /P12
- JP14 pad 2: 5.0V -> +5V
- JP15 pad 1: Net-(U7-AIN0) -> /P14
- JP15 pad 2: 3.3V -> +5V
- JP15 pad 4: Net-(U7-AIN1) -> /P15
- JP15 pad 5: 3.3V -> +5V
- JP2 pad 2: 3.3V -> +5V
- JP2 pad 3: Net-(U5-AIN0) -> /Ain0
- JP2 pad 5: 3.3V -> +5V
- JP2 pad 6: Net-(U5-AIN1) -> /Ain1
- JP3 pad 1: 5.0V -> +5V
- JP3 pad 3: /SDA -> /SDA_A
- JP3 pad 4: /SCL -> /SCL_A
- JP4 pad 1: 5.0V -> +5V
- JP4 pad 3: /SDA -> /SDA_A
- JP4 pad 4: /SCL -> /SCL_A
- JP5 pad 1: Net-(JP9-Pad1) -> Net-(D3-A)
- JP5 pad 2: VCC -> +3.3V
- JP7 pad 1: Net-(U2-EnB) -> Net-(U2-VREF)
- JP7 pad 2: 5.0V -> +5V
- JP8 pad 1: Net-(U2-EnA) -> Net-(U3-VREF)
- JP8 pad 2: 5.0V -> +5V
- R12 pad 5: Net-(J13-Pin_1) -> /P12
- R12 pad 6: Net-(J13-Pin_2) -> /P13
- R12 pad 7: Net-(J13-Pin_3) -> /P14
- R12 pad 8: Net-(J13-Pin_4) -> /P15
- R2 pad 3: /SCL -> /SCL_A
- R2 pad 4: /SDA -> /SDA_A
- R2 pad 5: 5.0V -> +3.3V
- R2 pad 6: 5.0V -> +3.3V
- R29 pad 1: Net-(LED1-PadC) -> Net-(D1-K)
- R5 pad 1: Net-(LED2-PadC) -> GND
- R5 pad 2: GND -> Net-(U2-ISEN)
- SJ_A0 pad 1: 5.0V -> +5V
- SJ_A1 pad 1: 5.0V -> +5V
- SJ_A2 pad 1: 5.0V -> +5V
- SJ_A3 pad 1: 5.0V -> +5V
- SJ_A4 pad 1: 5.0V -> +5V
- SJ_A5 pad 1: 5.0V -> +5V
- U1 pad 26: /SCL -> /SCL_B
- U1 pad 27: /SDA -> /SDA_B
- U1 pad 28: 5.0V -> +5V
- U2 pad : GND -> (no net)
- U2 pad 2: unconnected-(U2-SENSE_A-Pad2) -> /P0
- U2 pad 3: unconnected-(U2-NC-Pad3) -> /P1
- U2 pad 4: Net-(D2-A) -> Net-(U2-VREF)
- U2 pad 5: Net-(D4-A) -> VCC
- U2 pad 6: VCC -> Net-(U2-OUT1)
- U2 pad 7: /P3 -> Net-(U2-ISEN)
- U2 pad 8: Net-(U2-EnA) -> Net-(U2-OUT2)
- U2 pad 9: /P2 -> GND
- U3 pad : GND -> (no net)
- U3 pad 2: unconnected-(U3-SENSE_A-Pad2) -> /P2
- U3 pad 3: unconnected-(U3-NC-Pad3) -> /P3
- U3 pad 4: Net-(D10-A) -> Net-(U3-VREF)
- U3 pad 5: Net-(D12-A) -> VCC
- U3 pad 6: VCC -> Net-(U3-OUT1)
- U3 pad 7: /P7 -> Net-(U3-ISEN)
- U3 pad 8: Net-(U3-EnA) -> Net-(U3-OUT2)
- U3 pad 9: /P6 -> GND
- U4 pad : GND -> (no net)
- U4 pad 2: unconnected-(U4-SENSE_A-Pad2) -> /P4
- U4 pad 3: unconnected-(U4-NC-Pad3) -> /P5
- U4 pad 4: Net-(D18-A) -> Net-(U4-VREF)
- U4 pad 5: Net-(D20-A) -> VCC
- U4 pad 6: VCC -> Net-(U4-OUT1)
- U4 pad 7: /P11 -> Net-(U4-ISEN)
- U4 pad 8: Net-(U4-EnA) -> Net-(U4-OUT2)
- U4 pad 9: /P10 -> GND
- U5 pad 1: GND -> VCC
- U5 pad 2: unconnected-(U5-ALERT/RDY-Pad2) -> GND
- U5 pad 3: GND -> +5V
- U6 pad 1: 3.3V -> /SDA_B
- U6 pad 2: unconnected-(U6-ALERT/RDY-Pad2) -> GND
- U6 pad 3: GND -> +3.3V
- U6 pad 4: Net-(U6-AIN0) -> /SDA_A
- U6 pad 5: Net-(U6-AIN1) -> /SCL_A
- U6 pad 7: Net-(U6-AIN3) -> +5V
- U6 pad 8: 3.3V -> /SCL_B
- U7 pad 1: /SCL -> /SCL_B
- U7 pad 10: /SDA -> /In1
- U7 pad 2: unconnected-(U7-ALERT/RDY-Pad2) -> /SDA_B
- U7 pad 4: Net-(U7-AIN0) -> GND
- U7 pad 5: Net-(U7-AIN1) -> GND
- U7 pad 7: Net-(U7-AIN3) -> unconnected-(U7-NC-Pad7)
- U7 pad 8: 3.3V -> GND
- U7 pad 9: /SCL -> GND
- U8 pad 1: VCC -> Net-(R9-Pad1)
- U8 pad 3: 5.0V -> GND
Routing:
- net +5V: track 0.00 -> 705.5 mm, vias 0 -> 12
- net GND: track 625.3 -> 66.1 mm, vias 261 -> 123
- net 5.0V: track 198.2 -> 0.00 mm, vias 8 -> 0
- net 3.3V: track 162.1 -> 0.00 mm, vias 6 -> 0
- net VCC: track 386.7 -> 237.3 mm, vias 16 -> 0
- net /SDA_B: track 0.00 -> 140.9 mm, vias 0 -> 6
- net /SCL_B: track 0.00 -> 127.6 mm, vias 0 -> 6
- net /SCL: track 104.5 -> 0.00 mm, vias 7 -> 0
- net /SDA: track 100.4 -> 0.00 mm, vias 5 -> 0
- net Net-(U6-AIN3): track 89.3 -> 0.00 mm, vias 1 -> 0
- net Net-(U6-OE): track 89.2 -> 8.83 mm, vias 1 -> 0
- net +3.3V: track 0.00 -> 74.6 mm, vias 0 -> 4
- net /SDA_A: track 0.00 -> 70.8 mm, vias 0 -> 1
- net /SCL_A: track 0.00 -> 68.4 mm, vias 0 -> 3
- net /P5: track 4.00 -> 66.5 mm, vias 0 -> 2
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Other:
- board size 69.2 x 55.6 mm -> 63 x 79.3 mm
- board text added: "5V+"
- board text added: "ANALOG"
- board text added: "I2C->"
- board text added: "Water Quality Control"
- board text removed: "(Open=0/Closed=1)"
- board text removed: "1+"
- board text removed: "16 x 12-bit PWM"
- board text removed: "16-Channel 12-Bit PWM Driver"
- board text removed: "3-5V"
- board text removed: "40-1000Hz"
- board text removed: "6V Max"
- board text removed: "C2"
- board text removed: "Freq.:"
- board text removed: "I2C Address"
- board text removed: "Logic:"
- board text removed: "PCA9685"
- board text removed: "Terminal block is"
- board text removed: "Use V+ for servo supply"
- board text removed: "V+:"
- board text removed: "VCC:"
- board text removed: "adafruit!"
- board text removed: "pins are not!"
- board text removed: "protected. Side breakout"
- board text removed: "reverse polarity"
