File: Rev0/Rev0.kicad_pcb (KiCad board)
At the start: 2 copper layers, 63 x 79.3 mm, 137 parts, among them J1 TERMBLOCK_1X2, J10 TERMBLOCK_1X2, J11 TERMBLOCK_1X2, J12 TERMBLOCK_1X2, J13 TERMBLOCK_1X2, J19 TERMBLOCK_1X2, J2 QWIIC_RIGHT_ANGLE, J20 TERMBLOCK_1X2, J21 TERMBLOCK_1X2, J22 TERMBLOCK_1X2, J23 TERMBLOCK_1X2, J24 TERMBLOCK_1X2, J25 TERMBLOCK_1X2, J26 TERMBLOCK_1X2, J28 Conn_01x02, J29 Conn_01x02, J3 QWIIC_RIGHT_ANGLE, J30 Conn_01x02, J31 Conn_01x02, J32 Conn_01x02, J33 Conn_01x02, J34 Conn_01x02, J35 Conn_01x02, J4 TERMBLOCK_1X2, J5 TERMBLOCK_1X2, J6 TERMBLOCK_1X2, J7 TERMBLOCK_1X2, J8 TERMBLOCK_1X2, J9 TERMBLOCK_1X2, Q1 AOD417, U1 PCA9685, U10 PC817, U11 PC817, U12 PC817, U13 PC817, U14 PC817, U15 PC817, U16 ADS1115IDGS, U17 ADS1115IDGS, U2 DRV8870DDA, U3 DRV8870DDA, U4 DRV8870DDA, U5 K7805-2000R3L, U6 TCA9406DC, U7 MCP23008-xSO, U8 PC817, U9 PC817

Commit message: .
Parts:
- removed the J10 at (142.2, 124.8)
- added G***: LOGO, Graphics:qr-WaterQualityControl, F.Cu at (148.5, 124.9)
- added R35: 3.9K, Resistor_SMD:R_0603_1608Metric, F.Cu at (151.0, 116.8)
- added R36: 10K, Resistor_SMD:R_0603_1608Metric, F.Cu at (153.4, 110.0)
- added R37: 1K, Resistor_SMD:R_0603_1608Metric, F.Cu at (153.4, 111.5)
- added R38: 1K, Resistor_SMD:R_0603_1608Metric, F.Cu at (153.4, 113.0)
- C11, C7, C9: value 0.1uF -> 0.1uF/35v
- JP1, JP12, JP13, JP14, JP15, JP2: value Conn_02x03 -> Header 2x3
- R1, R2: value 10k -> 10k/603x4
- R11: renamed from R13; value 220 -> 220/603x4
- R12: renamed from R11; value 220 -> 220/603x4
- R13: renamed from R14; value 220 -> 220/603x4
- R14: renamed from R12; value 220 -> 220/603x4
- R30: value 1.5k -> 2K; footprint Adafruit PCA9685 rev C:RESPACK_4X0603 -> Resistor_SMD:R_0603_1608Metric
- moved G*** 25.7 mm to (148.5, 124.9)
- moved R30 11.5 mm to (152.7, 107.7), turned to 90 degrees
- moved J10 9.24 mm to (140.2, 124.8)
- moved C4 3.92 mm to (151.0, 119.8)
- moved U17 3.92 mm to (147.3, 119.5)
- moved C3 2.03 mm to (128.9, 118.6)
- moved JP1 2.03 mm to (134.0, 124.6)
- moved JP2 2.03 mm to (128.9, 124.6)
- moved U16 2.03 mm to (132.9, 118.9)
- moved C13 1.36 mm to (161.7, 87.8)
- moved C2 1.36 mm to (152.7, 96.1)
- moved C6 1.36 mm to (156.9, 115.2)
- moved D2 1.36 mm to (155.2, 76.5)
- moved JP9 1.36 mm to (156.6, 115.2)
- moved R5 1.36 mm to (165.0, 80.7)
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- renumbered J11 to J10
Connections:
- J10 pad 1: /Ain5 -> /Ain4
- R29 pad 1: Net-(D1-K) -> GND
- R29 pad 2: GND -> Net-(D1-K)
- R3 pad 1: /OE -> GND
- R3 pad 2: GND -> /OE
- R30 pad 1: /Ain4 -> /Ain5
- R30 pad 2: /Ain5 -> GND
- R31 pad 1: Net-(D2-A) -> GND
- R31 pad 2: GND -> Net-(D2-A)
- R33 pad 1: /SCL_B -> +5V
- R33 pad 2: +5V -> /SCL_B
- R34 pad 1: /SDA_B -> +5V
- R34 pad 2: +5V -> /SDA_B
- R4 pad 1: Net-(D3-K) -> GND
- R4 pad 2: GND -> Net-(D3-K)
Routing:
- net +5V: track 705.5 -> 748.7 mm
- net GND: track 66.1 -> 83.5 mm, vias 123 -> 127
- net /Ain7: track 41.4 -> 46.3 mm
- net /Ain4: track 17.0 -> 14.9 mm
- net VCC: track 237.3 -> 239.3 mm
- net Net-(U3-OUT1): track 8.81 -> 10.2 mm
- net Net-(U3-OUT2): track 7.48 -> 8.83 mm
- net Net-(U2-OUT2): track 7.47 -> 8.83 mm
- net Net-(U4-OUT2): track 7.48 -> 8.84 mm
- net Net-(U2-OUT1): track 8.78 -> 10.1 mm
- net Net-(U4-OUT1): track 8.82 -> 10.2 mm
- net /SDA_B: track 140.9 -> 142.0 mm
- net /A4: track 17.3 -> 18.3 mm
- net /Out4: track 17.3 -> 16.4 mm
- net /Ain5: track 18.2 -> 17.4 mm
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Other:
- board text added: "INPUT1"
- board text added: "INPUT2"
- board text added: "INPUT3"
- board text added: "INPUT4"
- board text added: "LEVEL1"
- board text added: "LEVEL2"
- board text added: "MOTOR1"
- board text added: "MOTOR2"
- board text added: "MOTOR3"
- board text added: "MOTOR4"
- board text added: "MOTOR5"
- board text added: "MOTOR6"
- board text added: "OUTPUT1"
- board text added: "OUTPUT2"
- board text added: "OUTPUT3"
- board text added: "OUTPUT4"
- board text added: "TEMP"

Commit message: .
Parts:
- R21, R23, R25, R27: value 750 -> 200
- R35: value 3.9K -> 270
Changed lines of the file:
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@@
         (effects (font (size 1 1) (thickness 0.15)))
     )
-    (fp_text value "3.9K" (at 0 1.43 90) (layer "F.Fab")
+    (fp_text value "270" (at 0 1.43 90) (layer "F.Fab")
         (effects (font (size 1 1) (thickness 0.15)))
     )
@@
         (effects (font (size 1 1) (thickness 0.15)))
     )
-    (fp_text value "750" (at 0 1.43 90) (layer "F.Fab")
+    (fp_text value "200" (at 0 1.43 90) (layer "F.Fab")
         (effects (font (size 1 1) (thickness 0.15)))
     )
@@
         (effects (font (size 1 1) (thickness 0.15)))
     )
-    (fp_text value "750" (at 0 1.43 90) (layer "F.Fab")
+    (fp_text value "200" (at 0 1.43 90) (layer "F.Fab")
         (effects (font (size 1 1) (thickness 0.15)))
     )
@@
         (effects (font (size 1 1) (thickness 0.15)))
     )
-    (fp_text value "750" (at 0 1.43 90) (layer "F.Fab")
+    (fp_text value "200" (at 0 1.43 90) (layer "F.Fab")
         (effects (font (size 1 1) (thickness 0.15)))
     )
@@
         (effects (font (size 1 1) (thickness 0.15)))
     )
-    (fp_text value "750" (at 0 1.43 90) (layer "F.Fab")
+    (fp_text value "200" (at 0 1.43 90) (layer "F.Fab")
         (effects (font (size 1 1) (thickness 0.15)))
     )
@@
     (fp_arc (start 0.508 2.413) (mid -0.569631 1.966631) (end -1.016 0.889)
       (stroke (width 0.254) (type solid)) (layer "B.SilkS"))
-    (fp_arc (start 8.229048 7.764478) (mid 9.052753 7.42388) (end 9.9441 7.42442)
+    (fp_arc (start 8.229048 7.764478) (mid 9.052754 7.423879) (end 9.9441 7.42442)
       (stroke (width 0.254) (type solid)) (layer "B.SilkS"))
     (fp_arc (start 8.234536 6.260553) (mid 9.129375 4.989852) (end 10.21588 3.87858)
@@
     (fp_arc (start 9.042459 6.381222) (mid 10.012997 5.890291) (end 11.06932 5.63118)
       (stroke (width 0.254) (type solid)) (layer "B.SilkS"))
-    (fp_arc (start 10.153621 6.316813) (mid 10.819745 6.177299) (end 11.49604 6.10108)
+    (fp_arc (start 10.153621 6.316813) (mid 10.819744 6.177296) (end 11.49604 6.10108)
       (stroke (width 0.254) (type solid)) (layer "B.SilkS"))
     (fp_arc (start 10.255067 3.840987) (mid 11.121885 3.322842) (end 12.12088 3.175)
@@
     (fp_arc (start 12.319 -0.635) (mid 13.396631 -0.188631) (end 13.843 0.889)
       (stroke (width 0.254) (type solid)) (layer "B.SilkS"))
-    (fp_arc (start 12.6365 3.172934) (mid 12.92792 3.230905) (end 13.17498 3.39598)
+    (fp_arc (start 12.6365 3.172934) (mid 12.927926 3.230899) (end 13.17498 3.39598)
       (stroke (width 0.254) (type solid)) (layer "B.SilkS"))
     (fp_arc (start 13.27787 5.527066) (mid 12.666712 5.829464) (end 12.0142 6.02742)
       (stroke (width 0.254) (type solid)) (layer "B.SilkS"))
-    (fp_arc (start 13.718022 1.77772) (mid 14.092522 2.33979) (end 14.224 3.00228)
+    (fp_arc (start 13.718022 1.77772) (mid 14.092534 2.33979) (end 14.224 3.00228)
       (stroke (width 0.254) (type solid)) (layer "B.SilkS"))
-    (fp_arc (start 13.776451 2.089441) (mid 14.108184 2.587709) (end 14.224 3.175)
+    (fp_arc (start 13.776451 2.089441) (mid 14.108196 2.587709) (end 14.224 3.175)
       (stroke (width 0.254) (type solid)) (layer "B.SilkS"))
     (fp_arc (start 13.843 0.889) (mid 13.396631 1.966631) (end 12.319 2.413)
       (stroke (width 0.254) (type solid)) (layer "B.SilkS"))
-    (fp_arc (start 13.933527 4.300844) (mid 12.739662 5.103149) (end 11.3792 5.57022)
+    (fp_arc (start 13.933527 4.300844) (mid 12.739664 5.103156) (end 11.3792 5.57022)
       (stroke (width 0.254) (type solid)) (layer "B.SilkS"))
     (fp_arc (start 13.94714 3.45186) (mid 13.587204 3.599468) (end 13.22832 3.44932)
       (stroke (width 0.254) (type solid)) (layer "B.SilkS"))
-    (fp_arc (start 13.955743 2.395289) (mid 14.154815 2.694956) (end 14.224 3.048)
+    (fp_arc (start 13.955743 2.395289) (mid 14.154803 2.694956) (end 14.224 3.048)
       (stroke (width 0.254) (type solid)) (layer "B.SilkS"))
     (fp_arc (start 14.143264 6.107415) (mid 13.349685 7.17762) (end 12.09294 7.62)
@@
     (fp_arc (start 14.328866 2.561046) (mid 14.49285 2.451478) (end 14.68628 2.413)
       (stroke (width 0.254) (type solid)) (layer "B.SilkS"))
-    (fp_arc (start 14.344359 4.449235) (mid 13.859877 5.026778) (end 13.28928 5.51942)
+    (fp_arc (start 14.344359 4.449235) (mid 13.859875 5.026775) (end 13.28928 5.51942)
       (stroke (width 0.254) (type solid)) (layer "B.SilkS"))
-    (fp_arc (start 14.35024 4.826757) (mid 14.339076 5.167151) (end 14.29004 5.50418)
+    (fp_arc (start 14.35024 4.826757) (mid 14.339075 5.167151) (end 14.29004 5.50418)
       (stroke (width 0.254) (type solid)) (layer "B.SilkS"))
-    (fp_arc (start 14.68628 2.411388) (mid 14.844363 2.442831) (end 14.97838 2.53238)
+    (fp_arc (start 14.68628 2.411388) (mid 14.844369 2.442825) (end 14.97838 2.53238)
       (stroke (width 0.254) (type solid)) (layer "B.SilkS"))
     (fp_arc (start 14.730126 3.530099) (mid 14.751792 3.304011) (end 14.81582 3.0861)
       (stroke (width 0.254) (type solid)) (layer "B.SilkS"))
-    (fp_arc (start 14.859445 3.404629) (mid 14.925626 3.074154) (end 15.113 2.794)
+    (fp_arc (start 14.859445 3.404629) (mid 14.92562 3.074148) (end 15.113 2.794)
       (stroke (width 0.254) (type solid)) (layer "B.SilkS"))
     (fp_arc (start 14.932206 4.285679) (mid 14.782902 3.921185) (end 14.732 3.5306)
       (stroke (width 0.254) (type solid)) (layer "B.SilkS"))
-    (fp_arc (start 15.111212 2.665208) (mid 15.275779 2.698133) (end 15.41526 2.79146)
+    (fp_arc (start 15.111212 2.665208) (mid 15.275768 2.698145) (end 15.41526 2.79146)
       (stroke (width 0.254) (type solid)) (layer "B.SilkS"))
-    (fp_arc (start 15.38866 2.763954) (mid 15.702814 3.271585) (end 15.7988 3.8608)
+    (fp_arc (start 15.38866 2.763954) (mid 15.702828 3.271585) (end 15.7988 3.8608)
       (stroke (width 0.254) (type solid)) (layer "B.SilkS"))
     (fp_arc (start 15.67766 2.671387) (mid 16.007869 3.019303) (end 16.1798 3.4671)
       (stroke (width 0.254) (type solid)) (layer "B.SilkS"))
-    (fp_arc (start 15.708 5.025489) (mid 15.294548 4.762299) (end 14.986 4.3815)
+    (fp_arc (start 15.708 5.025489) (mid 15.294541 4.762306) (end 14.986 4.3815)
       (stroke (width 0.254) (type solid)) (layer "B.SilkS"))
-    (fp_arc (start 16.026073 2.665697) (mid 16.126536 2.671678) (end 16.22552 2.68986)
+    (fp_arc (start 16.026073 2.665697) (mid 16.126535 2.67168) (end 16.22552 2.68986)
       (stroke (width 0.254) (type solid)) (layer "B.SilkS"))
     (fp_arc (start 16.227503 2.690547) (mid 16.535892 2.788064) (end 16.80718 2.96418)
@@
     (fp_arc (start 16.559205 4.805934) (mid 16.306617 4.337511) (end 16.2052 3.81508)
       (stroke (width 0.254) (type solid)) (layer "B.SilkS"))
-    (fp_arc (start 16.831054 2.986026) (mid 17.063406 3.333768) (end 17.145 3.74396)
+    (fp_arc (start 16.831054 2.986026) (mid 17.063417 3.333768) (end 17.145 3.74396)
       (stroke (width 0.254) (type solid)) (layer "B.SilkS"))
     (fp_arc (start 17.009851 5.046864) (mid 16.968283 4.574521) (end 17.07388 4.11226)
       (stroke (width 0.254) (type solid)) (layer "B.SilkS"))
-    (fp_arc (start 17.144717 3.743513) (mid 17.126889 3.931265) (end 17.07388 4.11226)
+    (fp_arc (start 17.144717 3.743513) (mid 17.126897 3.931268) (end 17.07388 4.11226)
       (stroke (width 0.254) (type solid)) (layer "B.SilkS"))
   )
