File: Rev0/Rev0.kicad_pcb (KiCad board)
At the start: 2 copper layers, 63 x 79.3 mm, 141 parts, among them J1 TERMBLOCK_1X2, J10 TERMBLOCK_1X2, J12 TERMBLOCK_1X2, J13 TERMBLOCK_1X2, J19 TERMBLOCK_1X2, J2 QWIIC_RIGHT_ANGLE, J20 TERMBLOCK_1X2, J21 TERMBLOCK_1X2, J22 TERMBLOCK_1X2, J23 TERMBLOCK_1X2, J24 TERMBLOCK_1X2, J25 TERMBLOCK_1X2, J26 TERMBLOCK_1X2, J28 Conn_01x02, J29 Conn_01x02, J3 QWIIC_RIGHT_ANGLE, J30 Conn_01x02, J31 Conn_01x02, J32 Conn_01x02, J33 Conn_01x02, J34 Conn_01x02, J35 Conn_01x02, J4 TERMBLOCK_1X2, J5 TERMBLOCK_1X2, J6 TERMBLOCK_1X2, J7 TERMBLOCK_1X2, J8 TERMBLOCK_1X2, J9 TERMBLOCK_1X2, Q1 AOD417, U1 PCA9685, U10 PC817, U11 PC817, U12 PC817, U13 PC817, U14 PC817, U15 PC817, U16 ADS1115IDGS, U17 ADS1115IDGS, U2 DRV8870DDA, U3 DRV8870DDA, U4 DRV8870DDA, U5 K7805-2000R3L, U6 TCA9406DC, U7 MCP23008-xSO, U8 PC817, U9 PC817

Commit message: .
Parts:
- R35: value 270 -> 1k
- moved C17 6.38 mm to (157.8, 59.9), turned to 180 degrees
- moved R32 6.02 mm to (157.8, 58.3), turned to 180 degrees
- renumbered U17 to U16, U16 to U17
Connections:
- J10 pad 1: /Ain4 -> /Ain0
- J12 pad 1: /Ain6 -> /Ain2
- J13 pad 1: /Ain7 -> /Ain3
- JP1 pad 3: /Ain2 -> /Ain6
- JP1 pad 6: /Ain3 -> /Ain7
- JP2 pad 3: /Ain0 -> /Ain4
- JP2 pad 6: /Ain1 -> /Ain5
- R30 pad 1: /Ain5 -> /Ain1
- R32 pad 1: Net-(U6-OE) -> +3.3V
- R35 pad 2: /Ain4 -> /Ain0
- R36 pad 2: /Ain5 -> /Ain1
- R37 pad 2: /Ain6 -> /Ain2
- R38 pad 2: /Ain7 -> /Ain3
- U16 pad 4: /Ain4 -> /Ain0
- U16 pad 5: /Ain5 -> /Ain1
- U16 pad 6: /Ain6 -> /Ain2
- U16 pad 7: /Ain7 -> /Ain3
- U17 pad 4: /Ain0 -> /Ain4
- U17 pad 5: /Ain1 -> /Ain5
- U17 pad 6: /Ain2 -> /Ain6
- U17 pad 7: /Ain3 -> /Ain7
- U6 pad 6: Net-(U6-OE) -> +3.3V
- U7 pad 8: GND -> unconnected-(U7-INT-Pad8)
Routing:
- net /Ain7: track 46.3 -> 3.72 mm
- net /Ain3: track 3.72 -> 46.3 mm
- net /Ain6: track 40.5 -> 3.24 mm
- net /Ain2: track 3.24 -> 40.5 mm
- net /Ain5: track 17.4 -> 2.43 mm
- net /Ain1: track 2.43 -> 17.4 mm
- net +3.3V: track 74.6 -> 88.9 mm
- net /Ain4: track 14.9 -> 4.36 mm
- net /Ain0: track 4.36 -> 14.9 mm
- net Net-(U6-OE): track 8.83 -> 0.00 mm
- net +5V: track 748.7 -> 743.2 mm
- net GND: track 83.5 -> 88.7 mm, vias 127 -> 125
- net /SDA_A: track 70.8 -> 71.7 mm

Commit message: .
Parts:
- added G***: LOGO, Graphics:Hasatio_logo_micro, F.Cu at (145.8, 121.3)
- J1, J10, J12, J13, J19, J20, J21, J22, J23, J24, J25, J26, J4, J5, J6, J7, J8, J9: footprint Adafruit PCA9685 rev C:TERMBLOCK_1X2-3.5MM -> Connector_Phoenix_MC:PhoenixContact_MC_1,5_2-G-3.5_1x02_P3.50mm_Horizontal
- moved U$48 17.8 mm to (112.2, 143.7)
- moved J35 17.8 mm to (122.4, 137.2)
- moved U$e 17.8 mm to (174.4, 143.7)
- moved U17 17.6 mm to (133.4, 136.5)
- moved C3 17.6 mm to (129.4, 136.2)
- moved JP1 17.6 mm to (134.5, 142.2)
- moved JP2 17.6 mm to (129.4, 142.2)
- moved R30 17.0 mm to (151.3, 124.7)
- moved R36 17.0 mm to (152.2, 126.9)
- moved R37 17.0 mm to (152.2, 128.4)
- moved R38 17.0 mm to (152.2, 130.0)
- moved J26 16.3 mm to (118.3, 134.2)
- moved J34 15.4 mm to (122.4, 127.6)
- moved G*** 14.8 mm to (133.8, 126.7) (x2)
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- renumbered U$50 to U$e
Connections:
- J1 pad 1: GND -> Net-(Q1-D)
- J1 pad 2: Net-(Q1-D) -> GND
- J19 pad 1: /I1 -> +5V
- J19 pad 2: +5V -> /I1
- J20 pad 1: /I2 -> +5V
- J20 pad 2: +5V -> /I2
- J21 pad 1: /I3 -> +5V
- J21 pad 2: +5V -> /I3
- J22 pad 1: /I4 -> +5V
- J22 pad 2: +5V -> /I4
- J23 pad 1: /O1B -> /O1A
- J23 pad 2: /O1A -> /O1B
- J24 pad 1: /O2B -> /O2A
- J24 pad 2: /O2A -> /O2B
- J25 pad 1: /O3B -> /O3A
- J25 pad 2: /O3A -> /O3B
- J26 pad 1: /O4B -> /O4A
- J26 pad 2: /O4A -> /O4B
Routing:
- net +5V: track 743.2 -> 637.2 mm, vias 12 -> 20
- net VCC: track 239.3 -> 292.7 mm
- net GND: track 88.7 -> 132.6 mm, vias 125 -> 129
- net /Ain2: track 40.5 -> 13.4 mm
- net /SCL_B: track 127.2 -> 153.5 mm
- net /SDA_B: track 142.0 -> 159.3 mm
- net /O4A: track 22.3 -> 38.9 mm
- net /O4B: track 13.0 -> 28.9 mm
- net /O3A: track 20.8 -> 34.9 mm
- net /O3B: track 12.0 -> 25.2 mm
- net /Ain3: track 46.3 -> 33.3 mm
- net /P4: track 64.5 -> 76.6 mm
- net /P5: track 65.9 -> 78.0 mm
- net /O2B: track 10.5 -> 21.8 mm
- net /O2A: track 20.1 -> 31.1 mm
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Other:
- board size 63 x 79.3 mm -> 67.3 x 96.9 mm

Commit message: .
Parts:
- C5: footprint Capacitor_SMD:C_0603_1608Metric -> Capacitor_SMD:C_0805_2012Metric
- R11, R12, R13, R14: value 220/603x4 -> 220R/603x4
- R16, R18, R20, R9: value 750 -> 750R
- R21, R23, R25, R27: value 200 -> 200R
- R22, R24, R26, R28: value 100 -> 100R
- moved C5 0.39 mm to (154.2, 82.3)
Routing:
- net GND: track 132.6 -> 135.6 mm
- net /SCL_B: track 153.5 -> 152.3 mm
- net /SDA_B: track 159.3 -> 158.6 mm

Commit message: .
Changed lines of the file:
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@@
     (fp_arc (start 0.508 2.413) (mid -0.569631 1.966631) (end -1.016 0.889)
       (stroke (width 0.254) (type solid)) (layer "B.SilkS"))
-    (fp_arc (start 8.229048 7.764478) (mid 9.052754 7.423877) (end 9.9441 7.42442)
+    (fp_arc (start 8.229048 7.764478) (mid 9.052753 7.423878) (end 9.9441 7.42442)
       (stroke (width 0.254) (type solid)) (layer "B.SilkS"))
     (fp_arc (start 8.234536 6.260553) (mid 9.129375 4.989852) (end 10.21588 3.87858)
@@
     (fp_arc (start 9.042459 6.381222) (mid 10.012997 5.890291) (end 11.06932 5.63118)
       (stroke (width 0.254) (type solid)) (layer "B.SilkS"))
-    (fp_arc (start 10.153621 6.316813) (mid 10.819746 6.177305) (end 11.49604 6.10108)
+    (fp_arc (start 10.153621 6.316813) (mid 10.819745 6.177303) (end 11.49604 6.10108)
       (stroke (width 0.254) (type solid)) (layer "B.SilkS"))
     (fp_arc (start 10.255067 3.840987) (mid 11.121885 3.322842) (end 12.12088 3.175)
@@
     (fp_arc (start 12.319 -0.635) (mid 13.396631 -0.188631) (end 13.843 0.889)
       (stroke (width 0.254) (type solid)) (layer "B.SilkS"))
-    (fp_arc (start 12.6365 3.172934) (mid 12.92792 3.230905) (end 13.17498 3.39598)
+    (fp_arc (start 12.6365 3.172934) (mid 12.927926 3.230899) (end 13.17498 3.39598)
       (stroke (width 0.254) (type solid)) (layer "B.SilkS"))
     (fp_arc (start 13.27787 5.527066) (mid 12.666712 5.829464) (end 12.0142 6.02742)
       (stroke (width 0.254) (type solid)) (layer "B.SilkS"))
-    (fp_arc (start 13.718022 1.77772) (mid 14.092522 2.33979) (end 14.224 3.00228)
+    (fp_arc (start 13.718022 1.77772) (mid 14.092534 2.33979) (end 14.224 3.00228)
       (stroke (width 0.254) (type solid)) (layer "B.SilkS"))
-    (fp_arc (start 13.776451 2.089441) (mid 14.108184 2.587709) (end 14.224 3.175)
+    (fp_arc (start 13.776451 2.089441) (mid 14.108196 2.587709) (end 14.224 3.175)
       (stroke (width 0.254) (type solid)) (layer "B.SilkS"))
     (fp_arc (start 13.843 0.889) (mid 13.396631 1.966631) (end 12.319 2.413)
       (stroke (width 0.254) (type solid)) (layer "B.SilkS"))
-    (fp_arc (start 13.933527 4.300844) (mid 12.739662 5.103149) (end 11.3792 5.57022)
+    (fp_arc (start 13.933527 4.300844) (mid 12.739664 5.103156) (end 11.3792 5.57022)
       (stroke (width 0.254) (type solid)) (layer "B.SilkS"))
     (fp_arc (start 13.94714 3.45186) (mid 13.587204 3.599468) (end 13.22832 3.44932)
       (stroke (width 0.254) (type solid)) (layer "B.SilkS"))
-    (fp_arc (start 13.955743 2.395289) (mid 14.154815 2.694956) (end 14.224 3.048)
+    (fp_arc (start 13.955743 2.395289) (mid 14.154803 2.694956) (end 14.224 3.048)
       (stroke (width 0.254) (type solid)) (layer "B.SilkS"))
     (fp_arc (start 14.143264 6.107415) (mid 13.349685 7.17762) (end 12.09294 7.62)
@@
     (fp_arc (start 14.328866 2.561046) (mid 14.49285 2.451478) (end 14.68628 2.413)
       (stroke (width 0.254) (type solid)) (layer "B.SilkS"))
-    (fp_arc (start 14.344359 4.449235) (mid 13.859876 5.026777) (end 13.28928 5.51942)
+    (fp_arc (start 14.344359 4.449235) (mid 13.859873 5.026773) (end 13.28928 5.51942)
       (stroke (width 0.254) (type solid)) (layer "B.SilkS"))
-    (fp_arc (start 14.35024 4.826757) (mid 14.339076 5.167151) (end 14.29004 5.50418)
+    (fp_arc (start 14.35024 4.826757) (mid 14.339075 5.167151) (end 14.29004 5.50418)
       (stroke (width 0.254) (type solid)) (layer "B.SilkS"))
-    (fp_arc (start 14.68628 2.411388) (mid 14.844363 2.442831) (end 14.97838 2.53238)
+    (fp_arc (start 14.68628 2.411388) (mid 14.844369 2.442825) (end 14.97838 2.53238)
       (stroke (width 0.254) (type solid)) (layer "B.SilkS"))
     (fp_arc (start 14.730126 3.530099) (mid 14.751792 3.304011) (end 14.81582 3.0861)
       (stroke (width 0.254) (type solid)) (layer "B.SilkS"))
-    (fp_arc (start 14.859445 3.404629) (mid 14.925626 3.074154) (end 15.113 2.794)
+    (fp_arc (start 14.859445 3.404629) (mid 14.92562 3.074148) (end 15.113 2.794)
       (stroke (width 0.254) (type solid)) (layer "B.SilkS"))
     (fp_arc (start 14.932206 4.285679) (mid 14.782902 3.921185) (end 14.732 3.5306)
       (stroke (width 0.254) (type solid)) (layer "B.SilkS"))
-    (fp_arc (start 15.111212 2.665208) (mid 15.275779 2.698133) (end 15.41526 2.79146)
+    (fp_arc (start 15.111212 2.665208) (mid 15.275768 2.698145) (end 15.41526 2.79146)
       (stroke (width 0.254) (type solid)) (layer "B.SilkS"))
-    (fp_arc (start 15.38866 2.763954) (mid 15.702814 3.271585) (end 15.7988 3.8608)
+    (fp_arc (start 15.38866 2.763954) (mid 15.702828 3.271585) (end 15.7988 3.8608)
       (stroke (width 0.254) (type solid)) (layer "B.SilkS"))
     (fp_arc (start 15.67766 2.671387) (mid 16.007869 3.019303) (end 16.1798 3.4671)
       (stroke (width 0.254) (type solid)) (layer "B.SilkS"))
-    (fp_arc (start 15.708 5.025489) (mid 15.294548 4.762303) (end 14.986 4.3815)
+    (fp_arc (start 15.708 5.025489) (mid 15.294555 4.762296) (end 14.986 4.3815)
       (stroke (width 0.254) (type solid)) (layer "B.SilkS"))
-    (fp_arc (start 16.026073 2.665697) (mid 16.126536 2.671678) (end 16.22552 2.68986)
+    (fp_arc (start 16.026073 2.665697) (mid 16.126535 2.67168) (end 16.22552 2.68986)
       (stroke (width 0.254) (type solid)) (layer "B.SilkS"))
     (fp_arc (start 16.227503 2.690547) (mid 16.535892 2.788064) (end 16.80718 2.96418)
@@
     (fp_arc (start 16.559205 4.805934) (mid 16.306617 4.337511) (end 16.2052 3.81508)
       (stroke (width 0.254) (type solid)) (layer "B.SilkS"))
-    (fp_arc (start 16.831054 2.986026) (mid 17.063406 3.333768) (end 17.145 3.74396)
+    (fp_arc (start 16.831054 2.986026) (mid 17.063417 3.333768) (end 17.145 3.74396)
       (stroke (width 0.254) (type solid)) (layer "B.SilkS"))
     (fp_arc (start 17.009851 5.046864) (mid 16.968283 4.574521) (end 17.07388 4.11226)
       (stroke (width 0.254) (type solid)) (layer "B.SilkS"))
-    (fp_arc (start 17.144717 3.743513) (mid 17.126889 3.931265) (end 17.07388 4.11226)
+    (fp_arc (start 17.144717 3.743513) (mid 17.126897 3.931268) (end 17.07388 4.11226)
       (stroke (width 0.254) (type solid)) (layer "B.SilkS"))
   )
@@
   (segment (start 127.408357 111.924117) (end 126.872267 112.460207) (width 0.254) (layer "F.Cu") (net 105))
   (segment (start 125.235267 113.925781) (end 125.235267 114.762363) (width 0.254) (layer "F.Cu") (net 105))
-  (segment (start 126.037267 133.579306) (end 122.427401 137.189172) (width 0.508) (layer "F.Cu") (net 106))
+  (segment (start 126.037267 133.579306) (end 122.427401 137.189172) (width 0.254) (layer "F.Cu") (net 106))
   (segment (start 126.037267 114.344072) (end 126.140067 114.241272) (width 0.508) (layer "F.Cu") (net 106))
-  (segment (start 126.037267 114.344072) (end 126.037267 133.579306) (width 0.508) (layer "F.Cu") (net 106))
+  (segment (start 126.037267 114.344072) (end 126.037267 133.579306) (width 0.254) (layer "F.Cu") (net 106))
   (segment (start 121.897401 137.719172) (end 122.427401 137.189172) (width 2.032) (layer "F.Cu") (net 106))
   (segment (start 118.277401 137.719172) (end 121.897401 137.719172) (width 2.032) (layer "F.Cu") (net 106))
