File: Rev0/Rev0.kicad_sch (KiCad schematic)
At the start: 98 parts, among them J1 TERMBLOCK_1X2, J10 TERMBLOCK_1X2, J11 TERMBLOCK_1X2, J13 Conn_01x04, J4 TERMBLOCK_1X2, J5 TERMBLOCK_1X2, J7 QWIIC_RIGHT_ANGLE, J7 TERMBLOCK_1X2, J8 TERMBLOCK_1X2, Q1 AOD417, U1 PCA9685, U2 L298P, U3 L298P, U4 L298P, U5 ADS1115IDGS, U6 ADS1115IDGS, U7 ADS1115IDGS, U8 L7805

Commit message: .
Parts:
- removed C2: 1000uF, Adafruit PCA9685 rev C:E3,5-8, symbol Adafruit PCA9685 rev C-eagle-import:CPOL-USE3.5-8
- removed D1, D10, D11, D12, D13, D14, D15, D16, D17, D18, D19, D2, D20, D21, D22, D23, D24, D25, D3, D4, D5, D6, D7, D8, D9: M7, Diode_SMD:D_SMA, symbol PCM_Diode_AKL:M7
- removed FID1, FID2: FIDUCIAL{dblquote}{dblquote}, Adafruit PCA9685 rev C:FIDUCIAL_1MM, symbol Adafruit PCA9685 rev C-eagle-import:FIDUCIAL{dblquote}{dblquote}
- removed J13: Conn_01x04, Connector_PinHeader_2.54mm:PinHeader_1x04_P2.54mm_Vertical, symbol Connector_Generic:Conn_01x04
- removed JP1 (x7): JUMPER-SMT_2_NC_TRACE_SILK, OLIMEX_Jumpers-FP:SJ_Closed, symbol SparkFun ESP32 Thing Plus C-eagle-import:JUMPER-SMT_2_NC_TRACE_SILK
- removed JP16, JP5, JP6: ~, Adafruit PCA9685 rev C:3X02, symbol Adafruit PCA9685 rev C-eagle-import:HEADER-3X02
- removed LED1: GREEN, Adafruit PCA9685 rev C:CHIPLED_0805_NOOUTLINE, symbol Adafruit PCA9685 rev C-eagle-import:LED0805_NOOUTLINE
- removed LED2: RED, Adafruit PCA9685 rev C:CHIPLED_0805_NOOUTLINE, symbol Adafruit PCA9685 rev C-eagle-import:LED0805_NOOUTLINE
- removed R5: 470, Adafruit PCA9685 rev C:_0805MP, symbol Adafruit PCA9685 rev C-eagle-import:RESISTOR_0805MP
- removed U$47, U$48, U$49, U$50: MOUNTINGHOLE2.5, Adafruit PCA9685 rev C:MOUNTINGHOLE_2.5_PLATED, symbol Adafruit PCA9685 rev C-eagle-import:MOUNTINGHOLE2.5
- removed U2, U3, U4: L298P, symbol Driver_Motor:L298P
- removed U7: ADS1115IDGS, Package_SO:TSSOP-10_3x3mm_P0.5mm, symbol Analog_ADC:ADS1115IDGS
- removed U8: L7805, PCM_Package_TO_SOT_SMD_AKL:TO-252-3_TabPin2, symbol Regulator_Linear:L7805
- added C10, C11, C16, C17, C18: 0.1uF, Capacitor_SMD:C_0603_1608Metric, symbol Adafruit PCA9685 rev C-eagle-import:CAP_CERAMIC0805-NOOUTLINE
- added C12: 10uF, Capacitor_SMD:C_0603_1608Metric, symbol Adafruit PCA9685 rev C-eagle-import:CAP_CERAMIC0805-NOOUTLINE
- added C13, C14, C15: 47uF/35v, Capacitor_THT:C_Radial_D6.3mm_H11.0mm_P2.50mm, symbol Device:C_Polarized_Small
- added C2: 1000uF/35v, Capacitor_THT:C_Radial_D10.0mm_H20.0mm_P5.00mm, symbol Device:C_Polarized_Small
- added D1: GREEN, LED_SMD:LED_0603_1608Metric, symbol Device:LED
- added D2: Z1SMA4740, Diode_SMD:D_SMA, symbol Diode:Z1SMAxxx
- added D3: RED, LED_SMD:LED_0603_1608Metric, symbol Device:LED
- added J10, J11, J12, J13, J19, J20, J21, J22, J23, J24, J25, J26: TERMBLOCK_1X2, Adafruit PCA9685 rev C:TERMBLOCK_1X2-3.5MM, symbol Adafruit PCA9685 rev C-eagle-import:TERMBLOCK_1X2
- added J28, J29, J30, J31, J32, J33, J34, J35: Conn_01x02, Connector_PinHeader_2.54mm:PinHeader_1x02_P2.54mm_Vertical, symbol Connector_Generic:Conn_01x02
- added JP1 (x4): JUMPER-SMT_2_NC_TRACE_SILK, OLIMEX_Jumpers-FP:SJ_Closed, symbol SparkFun ESP32 Thing Plus C-eagle-import:JUMPER-SMT_2_NC_TRACE_SILK
- added JP12, JP13, JP14: Header 2x3, Adafruit PCA9685 rev C:3X02, symbol Adafruit PCA9685 rev C-eagle-import:HEADER-3X02
- added R10, R15, R17, R19, R32, R33, R34, R8: 10K, Resistor_SMD:R_0603_1608Metric, symbol Adafruit PCA9685 rev C-eagle-import:RESISTOR0805_NOOUTLINE
- added R16, R18, R20, R21, R23, R25, R27, R9: 750, Resistor_SMD:R_0603_1608Metric, symbol Adafruit PCA9685 rev C-eagle-import:RESISTOR0805_NOOUTLINE
- added R22, R24, R26, R28: 100, Resistor_SMD:R_0603_1608Metric, symbol Adafruit PCA9685 rev C-eagle-import:RESISTOR0805_NOOUTLINE
- added R29: 1k, Resistor_SMD:R_0603_1608Metric, symbol Adafruit PCA9685 rev C-eagle-import:RESISTOR_0805MP
- added R30: 1.5k 603x4, Adafruit PCA9685 rev C:RESPACK_4X0603, symbol Adafruit PCA9685 rev C-eagle-import:RESISTOR_4PACK
- added R31: 100k, Resistor_SMD:R_0603_1608Metric, symbol Adafruit PCA9685 rev C-eagle-import:RESISTOR0805_NOOUTLINE
- added R5, R6, R7: 250m/1w, Resistor_SMD:R_1206_3216Metric, symbol Adafruit PCA9685 rev C-eagle-import:RESISTOR0805_NOOUTLINE
- added U10, U11, U12, U13, U14, U15, U8, U9: PC817, Package_DIP:DIP-4_W7.62mm_SMDSocket_SmallPads, symbol Isolator:PC817
- added U2: K7805-2000R3L, Converter_DCDC:Converter_DCDC_RECOM_R-78HB-0.5L_THT, symbol Regulator_Switching:R-78B5.0-2.0
- added U2, U3, U4: DRV8870DDA, Package_SO:Texas_HTSOP-8-1EP_3.9x4.9mm_P1.27mm_EP2.95x4.9mm_Mask2.4x3.1mm_ThermalVias, symbol Driver_Motor:DRV8870DDA
- added U6: TCA9406DC, PCM_Package_SO_AKL:SSOP-8_2.95x2.8mm_P0.65mm, symbol Interface:TCA9406DC
- added U7: MCP23008-xSO, Package_SO:SOIC-18W_7.5x11.6mm_P1.27mm, symbol Interface_Expansion:MCP23008-xSO
- C1: footprint Adafruit PCA9685 rev C:0805-NO -> Capacitor_SMD:C_0603_1608Metric
- C3, C4, C8, C9: value 1.0uF -> 0.1uF; footprint Adafruit PCA9685 rev C:0805-NO -> Capacitor_SMD:C_0603_1608Metric
- C5: value 1.0uF -> 10uF/35v; footprint Adafruit PCA9685 rev C:0805-NO -> Capacitor_SMD:C_0603_1608Metric
- C6, C7: value 10uF -> 0.1uF; footprint Adafruit PCA9685 rev C:0805-NO -> Capacitor_SMD:C_0603_1608Metric
- JP1, SJ_A0, SJ_A1, SJ_A2, SJ_A3, SJ_A4, SJ_A5: now left out of the parts list
- JP1, JP15, JP2: value ~ -> Header 2x3
- R1, R2: value 10K -> 10k 603x4
- R3: footprint Adafruit PCA9685 rev C:0805-NO -> Resistor_SMD:R_0603_1608Metric
- R4: footprint Adafruit PCA9685 rev C:_0805MP -> Resistor_SMD:R_0603_1608Metric
- renumbered J8 to J6, J11 to J8, J10 to J9
Connections:
- net GND: now also J1.1, J4.2, J5.2, J6.2, J7.2, J8.2, J9.2, U6.1 (ADDR), C10.2, C11.2, C12.2, C13.2, C14.2, C15.2, C16.2, C17.2, C18.2, C2.2, J10.2, J11.2, J12.2, J13.2, JP12.3, JP12.6, JP13.3, JP13.6, JP14.3, JP14.6, R29.2, R31.2, R32.2, R5.1, R6.1, R7.1, U10.2, U10.3, U11.2, U11.3, U12.2, U12.3, U13.2, U13.3, U14.2, U14.3, U15.2, U15.3, U2.1 (GND), U2.2 (GND), U2.9 (GND), U3.1 (GND), U3.9 (GND), U4.1 (GND), U4.9 (GND), U6.2 (GND), U7.3 (A2), U7.4 (A1), U7.5 (A0), U7.8 (INT), U7.9 (VSS), U8.2, U8.3, U9.2, U9.3; no longer J1.2, U5.1 (ADDR)
- net P0: now also U2.2 (IN2)
- net P1: now also U2.3 (IN1)
- net P10: now also JP13.1
- net P11: now also JP13.4
- net P2: now also U3.2 (IN2)
- net P3: now also U3.3 (IN1)
- net P4: now also U4.2 (IN2)
- net P5: now also U4.3 (IN1)
- net P8: now also JP12.1
- net P9: now also JP12.4
- net VCC: now also C5.1, C7.1, C9.1, C11.1, C13.1, C14.1, C15.1, C2.1, D2.1 (K), R30.5 (2), R30.6 (2), R30.7 (2), R30.8 (2), U2.1 (IN), U2.5 (VM), U3.5 (VM), U4.5 (VM); no longer C6.1, C8.1
- net at J7.1: now also U3.6 (OUT1)
- net at J6.1: now also U3.8 (OUT2)
- net P14: now reaches R12.7 (2)
- net P14: now also JP15.1
- net at J9.1: now also U4.6 (OUT1)
- net at J4.1: now also U2.8 (OUT2)
- net at J5.1: now also U2.6 (OUT1)
- net P15: now reaches JP15.4
- net P15: now also R12.8 (2)
- net Ain4: now reaches U6.4 (AIN0)
- net Ain4: now also J10.1, R30.1
- net Ain5: now reaches U6.5 (AIN1)
- net Ain5: now also J11.1, R30.2 (1)
- net P13: now reaches R12.6 (2)
- net P13: now also JP14.4
- net at JP1.1: now also U2.4 (VREF)
- net at J8.1: now also U4.8 (OUT2)
- net Ain0: now reaches JP2.3
- net Ain0: now also U5.4 (AIN0); no longer U5.6 (AIN2)
- net Ain1: now reaches JP2.6
- net Ain1: now also U5.5 (AIN1); no longer U5.7 (AIN3)
- net Ain2: now reaches JP1.3
- net Ain2: now also U5.6 (AIN2); no longer U5.4 (AIN0)
- net Ain3: now reaches JP1.6
- net Ain3: now also U5.7 (AIN3); no longer U5.5 (AIN1)
- net at Q1.3 (D): now also J1.2; no longer J1.1
- net at R4.1: now also D3.1 (K)
- net Ain6: now reaches U6.6 (AIN2)
- net Ain6: now also J12.1, R30.3 (1)
- net Ain7: now reaches U6.7 (AIN3)
- net Ain7: now also J13.1, R30.4 (1)
- net P12: now reaches R12.5 (2)
- net P12: now also JP14.1
- net 3.3V renamed +5V
- net +5V: now also C1.1, C6.1, C8.1, JP1.2, JP3.1, JP4.1, SJ_A0.1, SJ_A1.1, SJ_A2.1, SJ_A3.1, SJ_A4.1, SJ_A5.1, U1.28 (VDD), U5.1 (ADDR), C10.1, C12.1, C17.1, C18.1, J19.2, J20.2, J21.2, J22.2, J28.2 (Pin_2), J29.2 (Pin_2), J30.2 (Pin_2), J31.2 (Pin_2), JP1.2, JP1.2, JP1.2, JP12.2, JP12.5, JP13.2, JP13.5, JP14.2, JP14.5, R10.2, R15.2, R17.2, R19.2, R22.2, R24.2, R26.2, R28.2, R33.2, R34.2, R8.2, U2.3 (OUT), U6.7 (VCCB), U7.18 (VDD); no longer C5.1, J7.2, J7.2, U6.1 (ADDR)
- removed net 5.0V: C1.1, C7.1, C9.1, JP1.2, JP3.1, JP4.1, R2.5 (2), R2.6 (2), SJ_A0.1, SJ_A1.1, SJ_A2.1, SJ_A3.1, SJ_A4.1, SJ_A5.1, U1.28 (VDD)
- net SCL renamed SCL_A
- net SCL_A: now also U6.5 (SCL_A); no longer U1.26 (SCL), U5.10 (SCL), U6.10 (SCL)
- net SDA renamed SDA_A
- net SDA_A: now also U6.4 (SDA_A); no longer U1.27 (SDA), U5.9 (SDA), U6.9 (SDA)
- new net: R27.1, U15.1
- new net: R16.1, U9.1
- new net: R23.1, U13.1
- new net: R21.1, U12.1
- new net: R25.1, U14.1
- new net: R5.2, U2.7 (ISEN)
- new net: R6.2, U3.7 (ISEN)
- new net: R18.1, U10.1
- new net: R9.1, U8.1
- new net: JP1.1, U4.4 (VREF)
- new net: D2.2 (A), R31.1
- new net: D3.2 (A), JP1.1
- new net: R7.2, U4.7 (ISEN)
- new net: D1.2 (A), JP1.1
- new net: R32.1, U6.6 (OE)
- new net: JP1.1, U3.4 (VREF)
- new net: R15.1, U7.6 (~{RESET})
- new net: R20.1, U11.1
- new net: D1.1 (K), R29.1
- new net +3.3V: C16.1, J7.2, J7.2, JP1.2, R2.5 (2), R2.6 (2), U6.3 (VCCA)
- new net I1: J19.1, J28.1 (Pin_1), R9.2
- new net I2: J20.1, J29.1 (Pin_1), R16.2
- new net I3: J21.1, J30.1 (Pin_1), R18.2
- new net I4: J22.1, J31.1 (Pin_1), R20.2
- new net In1: R8.1, U7.10 (GP0), U8.4
- new net In2: R10.1, U7.11 (GP1), U9.4
- new net In3: R17.1, U10.4, U7.12 (GP2)
- new net In4: R19.1, U11.4, U7.13 (GP3)
- new net O1A: J23.2, J32.2 (Pin_2), U12.4
- new net O1B: J23.1, J32.1 (Pin_1), R22.1
- new net O2A: J24.2, J33.2 (Pin_2), U13.4
- new net O2B: J24.1, J33.1 (Pin_1), R24.1
- new net O3A: J25.2, J34.2 (Pin_2), U14.4
- new net O3B: J25.1, J34.1 (Pin_1), R26.1
- new net O4A: J26.2, J35.2 (Pin_2), U15.4
- new net O4B: J26.1, J35.1 (Pin_1), R28.1
- new net Out1: R21.2, U7.14 (GP4)
- new net Out2: R23.2, U7.15 (GP5)
- new net Out3: R25.2, U7.16 (GP6)
- new net Out4: R27.2, U7.17 (GP7)
- new net SCL_B: R33.1, U1.26 (SCL), U5.10 (SCL), U6.10 (SCL), U6.8 (SCL_B), U7.1 (SCL)
- new net SDA_B: R34.1, U1.27 (SDA), U5.9 (SDA), U6.1 (SDA_B), U6.9 (SDA), U7.2 (SDA)
Other:
- note added: "I2C transfer"
- note added: "Input/Output"
- note added: "Motor Control"
- note added: "Sensor"
- note removed: "Analog"
- note removed: "L298"
- title: PCA9685+L298 -> Water Quality Control
- moved on the sheet: C1, C3, C4, J1, J4, J5, J6, J7, J8, J9, JP1, JP2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

Commit message: .
Parts:
- R30: value 1.5k 603x4 -> 1k 603x4
Changed lines of the file:
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@@
       (effects (font (size 1.27 1.27)))
     )
-    (property "Value" "1.5k 603x4" (at 26.67 195.58 0)
+    (property "Value" "1k 603x4" (at 26.67 195.58 0)
       (effects (font (size 1.016 1.016) bold))
     )
@@
       (effects (font (size 1.27 1.27)))
     )
-    (property "Value" "1.5k 603x4" (at 26.67 200.66 0)
+    (property "Value" "1k 603x4" (at 26.67 200.66 0)
       (effects (font (size 1.016 1.016) bold))
     )
@@
       (effects (font (size 1.27 1.27)))
     )
-    (property "Value" "1.5k 603x4" (at 26.67 185.42 0)
+    (property "Value" "1k 603x4" (at 26.67 185.42 0)
       (effects (font (size 1.016 1.016) bold))
     )
@@
       (effects (font (size 1.27 1.27)))
     )
-    (property "Value" "1.5k 603x4" (at 26.67 190.5 0)
+    (property "Value" "1k 603x4" (at 26.67 190.5 0)
       (effects (font (size 1.016 1.016) bold))
     )

Commit message: .
Parts:
- removed J11: TERMBLOCK_1X2, Adafruit PCA9685 rev C:TERMBLOCK_1X2-3.5MM, symbol Adafruit PCA9685 rev C-eagle-import:TERMBLOCK_1X2
- removed R30: 1k 603x4, Adafruit PCA9685 rev C:RESPACK_4X0603, symbol Adafruit PCA9685 rev C-eagle-import:RESISTOR_4PACK
- added R30: 2K, Resistor_SMD:R_0603_1608Metric, symbol Adafruit PCA9685 rev C-eagle-import:RESISTOR0805_NOOUTLINE
- added R35: 270, Resistor_SMD:R_0603_1608Metric, symbol Adafruit PCA9685 rev C-eagle-import:RESISTOR0805_NOOUTLINE
- added R36: 10K, Resistor_SMD:R_0603_1608Metric, symbol Adafruit PCA9685 rev C-eagle-import:RESISTOR0805_NOOUTLINE
- added R37, R38: 1K, Resistor_SMD:R_0603_1608Metric, symbol Adafruit PCA9685 rev C-eagle-import:RESISTOR0805_NOOUTLINE
- C11, C7, C9: value 0.1uF -> 0.1uF/35v
- R1, R2: value 10k 603x4 -> 10k/603x4
- R11, R12, R13, R14: value 220 -> 220/603x4
- SJ_A0, SJ_A1, SJ_A2, SJ_A3, SJ_A4, SJ_A5: now in the parts list
Connections:
- net +5V: now also R33.1, R34.1, R35.1; no longer R33.2, R34.2
- net Ain4: now also R35.2
- net Ain5: now also R30.1, R36.2
- net Ain6: now also R37.2
- net Ain7: now also R38.2
- net GND: now also R29.1, R3.1, R31.1, R4.1, R30.2; no longer R29.2, R3.2, R31.2, R4.2
- net OE: now also R3.2; no longer R3.1
- net P0: now also R11.5 (2); no longer R13.5 (2)
- net P1: now also R11.6 (2); no longer R13.6 (2)
- net P10: now also R13.7 (2); no longer R14.7 (2)
- net P11: now also R13.8 (2); no longer R14.8 (2)
- net P12: now also R14.5 (2); no longer R12.5 (2)
- net P13: now also R14.6 (2); no longer R12.6 (2)
- net P14: now also R14.7 (2); no longer R12.7 (2)
- net P15: now also R14.8 (2); no longer R12.8 (2)
- net P2: now also R11.7 (2); no longer R13.7 (2)
- net P3: now also R11.8 (2); no longer R13.8 (2)
- net P4: now also R12.5 (2); no longer R11.5 (2)
- net P5: now also R12.6 (2); no longer R11.6 (2)
- net P6: now also R12.7 (2); no longer R11.7 (2)
- net P7: now also R12.8 (2); no longer R11.8 (2)
- net P8: now also R13.5 (2); no longer R14.5 (2)
- net P9: now also R13.6 (2); no longer R14.6 (2)
- net PWM0: now also R11.4 (1); no longer R13.4 (1)
- net PWM1: now also R11.3 (1); no longer R13.3 (1)
- net PWM10: now also R13.2 (1); no longer R14.2 (1)
- net PWM11: now also R13.1; no longer R14.1
- net PWM12: now also R14.4 (1); no longer R12.4 (1)
- net PWM13: now also R14.3 (1); no longer R12.3 (1)
- net PWM14: now also R14.2 (1); no longer R12.2 (1)
- net PWM15: now also R14.1; no longer R12.1
- net PWM2: now also R11.2 (1); no longer R13.2 (1)
- net PWM3: now also R11.1; no longer R13.1
- net PWM4: now also R12.4 (1); no longer R11.4 (1)
- net PWM5: now also R12.3 (1); no longer R11.3 (1)
- net PWM6: now also R12.2 (1); no longer R11.2 (1)
- net PWM7: now also R12.1; no longer R11.1
- net PWM8: now also R13.4 (1); no longer R14.4 (1)
- net PWM9: now also R13.3 (1); no longer R14.3 (1)
- net SCL_B: now also R33.2; no longer R33.1
- net SDA_B: now also R34.2; no longer R34.1
- net VCC: now also R36.1, R37.1, R38.1
- net at D2.2 (A): now also R31.2; no longer R31.1
- net at D3.1 (K): now also R4.2; no longer R4.1
- net at D1.1 (K): now also R29.2; no longer R29.1
Other:
- moved on the sheet: C13, C14, C15, R11A, R11B, R11C, R11D, R12A, R12B, R12C, R12D, R13A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

Commit message: .
Parts:
- R21, R23, R25, R27: value 750 -> 200
Changed lines of the file:
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@@
       (effects (font (size 1.27 1.27)))
     )
-    (property "Value" "750" (at 185.42 266.7 0)
+    (property "Value" "200" (at 185.42 266.7 0)
       (effects (font (size 1.016 1.016) bold))
     )
@@
       (effects (font (size 1.27 1.27)))
     )
-    (property "Value" "750" (at 86.36 266.7 0)
+    (property "Value" "200" (at 86.36 266.7 0)
       (effects (font (size 1.016 1.016) bold))
     )
@@
       (effects (font (size 1.27 1.27)))
     )
-    (property "Value" "750" (at 119.38 266.7 0)
+    (property "Value" "200" (at 119.38 266.7 0)
       (effects (font (size 1.016 1.016) bold))
     )
@@
       (effects (font (size 1.27 1.27)))
     )
-    (property "Value" "750" (at 152.4 266.7 0)
+    (property "Value" "200" (at 152.4 266.7 0)
       (effects (font (size 1.016 1.016) bold))
     )

Commit message: .
Parts:
- R35: value 270 -> 1k
Connections:
- net +3.3V: now also R32.1, U6.6 (OE)
- net Ain0: now also J10.1, R35.2, U6.4 (AIN0); no longer JP2.3, U5.4 (AIN0)
- net Ain1: now also R30.1, R36.2, U6.5 (AIN1); no longer JP2.6, U5.5 (AIN1)
- net Ain2: now also J12.1, R37.2, U6.6 (AIN2); no longer JP1.3, U5.6 (AIN2)
- net Ain3: now also J13.1, R38.2, U6.7 (AIN3); no longer JP1.6, U5.7 (AIN3)
- net Ain4: now also JP2.3, U5.4 (AIN0); no longer J10.1, R35.2, U6.4 (AIN0)
- net Ain5: now also JP2.6, U5.5 (AIN1); no longer R30.1, R36.2, U6.5 (AIN1)
- net Ain6: now also JP1.3, U5.6 (AIN2); no longer J12.1, R37.2, U6.6 (AIN2)
- net Ain7: now also JP1.6, U5.7 (AIN3); no longer J13.1, R38.2, U6.7 (AIN3)
- net GND: no longer U7.8 (INT)
Other:
- moved on the sheet: J10, J12, J13, JP1, JP2, R30, R35, R36, R37, R38, U5, U6

Commit message: .
Parts:
- J1, J10, J12, J13, J19, J20, J21, J22, J23, J24, J25, J26, J4, J5, J6, J7, J8, J9: footprint Adafruit PCA9685 rev C:TERMBLOCK_1X2-3.5MM -> Connector_Phoenix_MC:PhoenixContact_MC_1,5_2-G-3.5_1x02_P3.50mm_Horizontal
Connections:
- net +5V: now also J19.1, J20.1, J21.1, J22.1; no longer J19.2, J20.2, J21.2, J22.2
- net GND: now also J1.2; no longer J1.1
- net I1: now also J19.2; no longer J19.1
- net I2: now also J20.2; no longer J20.1
- net I3: now also J21.2; no longer J21.1
- net I4: now also J22.2; no longer J22.1
- net O1A: now also J23.1; no longer J23.2
- net O1B: now also J23.2; no longer J23.1
- net O2A: now also J24.1; no longer J24.2
- net O2B: now also J24.2; no longer J24.1
- net O3A: now also J25.1; no longer J25.2
- net O3B: now also J25.2; no longer J25.1
- net O4A: now also J26.1; no longer J26.2
- net O4B: now also J26.2; no longer J26.1
- net at Q1.3 (D): now also J1.1; no longer J1.2
Other:
- moved on the sheet: J1

Commit message: .
Parts:
- C5: footprint Capacitor_SMD:C_0603_1608Metric -> Capacitor_SMD:C_0805_2012Metric
- R11, R12, R13, R14: value 220/603x4 -> 220R/603x4
- R16, R18, R20, R9: value 750 -> 750R
- R21, R23, R25, R27: value 200 -> 200R
- R22, R24, R26, R28: value 100 -> 100R
Changed lines of the file:
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@@
       (effects (font (size 1.27 1.27)))
     )
-    (property "Value" "200" (at 185.42 266.7 0)
+    (property "Value" "200R" (at 185.42 266.7 0)
       (effects (font (size 1.016 1.016) bold))
     )
@@
       (effects (font (size 1.27 1.27)))
     )
-    (property "Value" "750" (at 134.62 236.22 0)
+    (property "Value" "750R" (at 134.62 236.22 0)
       (effects (font (size 1.016 1.016) bold))
     )
@@
       (effects (font (size 1.27 1.27)))
     )
-    (property "Value" "220/603x4" (at 227.33 95.25 0)
+    (property "Value" "220R/603x4" (at 227.33 95.25 0)
       (effects (font (size 1.016 1.016) bold))
     )
@@
       (effects (font (size 1.27 1.27)))
     )
-    (property "Value" "200" (at 86.36 266.7 0)
+    (property "Value" "200R" (at 86.36 266.7 0)
       (effects (font (size 1.016 1.016) bold))
     )
@@
       (effects (font (size 1.27 1.27)))
     )
-    (property "Value" "220/603x4" (at 227.33 64.77 0)
+    (property "Value" "220R/603x4" (at 227.33 64.77 0)
       (effects (font (size 1.016 1.016) bold))
     )
@@
       (effects (font (size 1.27 1.27)))
     )
-    (property "Value" "200" (at 119.38 266.7 0)
+    (property "Value" "200R" (at 119.38 266.7 0)
       (effects (font (size 1.016 1.016) bold))
     )
@@
       (effects (font (size 1.27 1.27)))
     )
-    (property "Value" "200" (at 152.4 266.7 0)
+    (property "Value" "200R" (at 152.4 266.7 0)
       (effects (font (size 1.016 1.016) bold))
     )
@@
       (effects (font (size 1.27 1.27)))
     )
-    (property "Value" "220/603x4" (at 270.51 85.09 0)
+    (property "Value" "220R/603x4" (at 270.51 85.09 0)
       (effects (font (size 1.016 1.016) bold))
     )
@@
       (effects (font (size 1.27 1.27)))
     )
-    (property "Value" "750" (at 167.64 236.22 0)
+    (property "Value" "750R" (at 167.64 236.22 0)
       (effects (font (size 1.016 1.016) bold))
     )
@@
       (effects (font (size 1.27 1.27)))
     )
-    (property "Value" "220/603x4" (at 227.33 44.45 0)
+    (property "Value" "220R/603x4" (at 227.33 44.45 0)
       (effects (font (size 1.016 1.016) bold))
     )
@@
       (effects (font (size 1.27 1.27)))
     )
-    (property "Value" "750" (at 101.6 236.22 0)
+    (property "Value" "750R" (at 101.6 236.22 0)
       (effects (font (size 1.016 1.016) bold))
     )
@@
       (effects (font (size 1.27 1.27)))
     )
-    (property "Value" "100" (at 284.48 269.875 0)
+    (property "Value" "100R" (at 284.48 269.875 0)
       (effects (font (size 1.016 1.016) bold))
     )
@@
       (effects (font (size 1.27 1.27)))
     )
-    (property "Value" "220/603x4" (at 227.33 34.29 0)
+    (property "Value" "220R/603x4" (at 227.33 34.29 0)
       (effects (font (size 1.016 1.016) bold))
     )
@@
       (effects (font (size 1.27 1.27)))
     )
-    (property "Value" "220/603x4" (at 270.51 95.25 0)
+    (property "Value" "220R/603x4" (at 270.51 95.25 0)
       (effects (font (size 1.016 1.016) bold))
     )
@@
       (effects (font (size 1.27 1.27)))
     )
-    (property "Value" "100" (at 294.64 269.875 0)
+    (property "Value" "100R" (at 294.64 269.875 0)
       (effects (font (size 1.016 1.016) bold))
     )
@@
       (effects (font (size 1.27 1.27)))
     )
-    (property "Footprint" "Capacitor_SMD:C_0603_1608Metric" (at 306.07 44.45 0)
+    (property "Footprint" "Capacitor_SMD:C_0805_2012Metric" (at 306.07 44.45 0)
       (effects (font (size 1.27 1.27)) hide)
     )
@@
       (effects (font (size 1.27 1.27)))
     )
-    (property "Value" "220/603x4" (at 227.33 85.09 0)
+    (property "Value" "220R/603x4" (at 227.33 85.09 0)
       (effects (font (size 1.016 1.016) bold))
     )
@@
       (effects (font (size 1.27 1.27)))
     )
-    (property "Value" "220/603x4" (at 270.51 105.41 0)
+    (property "Value" "220R/603x4" (at 270.51 105.41 0)
       (effects (font (size 1.016 1.016) bold))
     )
@@
       (effects (font (size 1.27 1.27)))
     )
-    (property "Value" "220/603x4" (at 227.33 105.41 0)
+    (property "Value" "220R/603x4" (at 227.33 105.41 0)
       (effects (font (size 1.016 1.016) bold))
     )
@@
       (effects (font (size 1.27 1.27)))
     )
-    (property "Value" "220/603x4" (at 227.33 54.61 0)
+    (property "Value" "220R/603x4" (at 227.33 54.61 0)
       (effects (font (size 1.016 1.016) bold))
     )
@@
       (effects (font (size 1.27 1.27)))
     )
-    (property "Value" "100" (at 279.4 269.875 0)
+    (property "Value" "100R" (at 279.4 269.875 0)
       (effects (font (size 1.016 1.016) bold))
     )
@@
       (effects (font (size 1.27 1.27)))
     )
-    (property "Value" "220/603x4" (at 270.51 34.29 0)
+    (property "Value" "220R/603x4" (at 270.51 34.29 0)
       (effects (font (size 1.016 1.016) bold))
     )
@@
       (effects (font (size 1.27 1.27)))
     )
-    (property "Value" "750" (at 200.66 236.22 0)
+    (property "Value" "750R" (at 200.66 236.22 0)
       (effects (font (size 1.016 1.016) bold))
     )
@@
       (effects (font (size 1.27 1.27)))
     )
-    (property "Value" "220/603x4" (at 270.51 74.93 0)
+    (property "Value" "220R/603x4" (at 270.51 74.93 0)
       (effects (font (size 1.016 1.016) bold))
     )
@@
       (effects (font (size 1.27 1.27)))
     )
-    (property "Value" "220/603x4" (at 227.33 74.93 0)
+    (property "Value" "220R/603x4" (at 227.33 74.93 0)
       (effects (font (size 1.016 1.016) bold))
     )
@@
       (effects (font (size 1.27 1.27)))
     )
-    (property "Value" "220/603x4" (at 270.51 44.45 0)
+    (property "Value" "220R/603x4" (at 270.51 44.45 0)
       (effects (font (size 1.016 1.016) bold))
     )
@@
       (effects (font (size 1.27 1.27)))
     )
-    (property "Value" "220/603x4" (at 270.51 64.77 0)
+    (property "Value" "220R/603x4" (at 270.51 64.77 0)
       (effects (font (size 1.016 1.016) bold))
     )
@@
       (effects (font (size 1.27 1.27)))
     )
-    (property "Value" "220/603x4" (at 270.51 54.61 0)
+    (property "Value" "220R/603x4" (at 270.51 54.61 0)
       (effects (font (size 1.016 1.016) bold))
     )
@@
       (effects (font (size 1.27 1.27)))
     )
-    (property "Value" "100" (at 289.56 269.875 0)
+    (property "Value" "100R" (at 289.56 269.875 0)
       (effects (font (size 1.016 1.016) bold))
     )

Commit message: .
Parts:
- R33, R34: value 10K -> 4k7
Changed lines of the file:
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@@
       (effects (font (size 1.27 1.27)))
     )
-    (property "Value" "10K" (at 372.11 101.6 0)
+    (property "Value" "4k7" (at 372.11 101.6 0)
       (effects (font (size 1.016 1.016) bold))
     )
@@
       (effects (font (size 1.27 1.27)))
     )
-    (property "Value" "10K" (at 372.11 96.52 0)
+    (property "Value" "4k7" (at 372.11 96.52 0)
       (effects (font (size 1.016 1.016) bold))
     )
