File: Rev1/Rev1.kicad_sch (KiCad schematic)
At the start: 131 parts, among them J1 TERMBLOCK_1X2, J10 TERMBLOCK_1X2, J12 TERMBLOCK_1X2, J13 TERMBLOCK_1X2, J19 TERMBLOCK_1X2, J20 TERMBLOCK_1X2, J21 TERMBLOCK_1X2, J22 TERMBLOCK_1X2, J23 TERMBLOCK_1X2, J24 TERMBLOCK_1X2, J25 TERMBLOCK_1X2, J26 TERMBLOCK_1X2, J28 Conn_01x02, J29 Conn_01x02, J30 Conn_01x02, J31 Conn_01x02, J32 Conn_01x02, J33 Conn_01x02, J34 Conn_01x02, J35 Conn_01x02, J4 TERMBLOCK_1X2, J5 TERMBLOCK_1X2, J6 TERMBLOCK_1X2, J7 QWIIC_RIGHT_ANGLE, J7 TERMBLOCK_1X2, J8 TERMBLOCK_1X2, J9 TERMBLOCK_1X2, Q1 AOD417, U1 PCA9685, U10 PC817, U11 PC817, U12 PC817, U13 PC817, U14 PC817, U15 PC817, U2 DRV8870DDA, U2 K7805-2000R3L, U3 DRV8870DDA, U4 DRV8870DDA, U5 ADS1115IDGS, U6 ADS1115IDGS, U6 TCA9406DC, U7 MCP23008-xSO, U8 PC817, U9 PC817

Commit message: .
Parts:
- removed U10, U11, U12, U13, U14, U15, U8, U9: PC817, Package_DIP:DIP-4_W7.62mm_SMDSocket_SmallPads, symbol Isolator:PC817
- added U10, U11, U12, U13, U14, U15, U8, U9: LTV-817S, PCM_Package_DIP_AKL:SMDIP-4_W9.53mm, symbol Isolator:LTV-817S
- renumbered R9 to R10, R10 to R9
Connections:
- net GND: now also U10.2, U10.3, U11.2, U11.3, U12.2, U12.3, U13.2, U13.3, U14.2, U14.3, U15.2, U15.3, U8.2, U8.3, U9.2, U9.3
- net In1: now also U8.1
- net In2: now also U9.1
- net In3: now also U10.1
- net In4: now also U11.1
- net O1A: now also U12.4
- net O2A: now also U13.4
- net O3A: now also U14.4
- net O4A: now also U15.4
- net at R27.1: now also U15.1
- net at R16.1: now also U9.4
- net at R23.1: now also U13.1
- net at R21.1: now also U12.1
- net at R25.1: now also U14.1
- net at R18.1: now also U10.4
- net at R10.1: now also U8.4
- net at R20.1: now also U11.4

Commit message: Update Rev1.kicad_sch
Parts:
- R29: value 1k -> 1k3
- R4: value 1k -> 750R
Changed lines of the file:
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@@
       (effects (font (size 1.27 1.27)))
     )
-    (property "Value" "1k" (at 400.05 237.49 0)
+    (property "Value" "750R" (at 400.05 237.49 0)
       (effects (font (size 1.016 1.016) bold))
     )
@@
       (effects (font (size 1.27 1.27)))
     )
-    (property "Value" "1k" (at 359.41 44.45 0)
+    (property "Value" "1k3" (at 359.41 44.45 0)
       (effects (font (size 1.016 1.016) bold))
     )
