File: Rev1/Rev1.kicad_sch (KiCad schematic)
At the start: 131 parts, among them J1 TERMBLOCK_1X2, J10 TERMBLOCK_1X2, J12 TERMBLOCK_1X2, J13 TERMBLOCK_1X2, J19 TERMBLOCK_1X2, J20 TERMBLOCK_1X2, J21 TERMBLOCK_1X2, J22 TERMBLOCK_1X2, J23 TERMBLOCK_1X2, J24 TERMBLOCK_1X2, J25 TERMBLOCK_1X2, J26 TERMBLOCK_1X2, J28 Conn_01x02, J29 Conn_01x02, J30 Conn_01x02, J31 Conn_01x02, J32 Conn_01x02, J33 Conn_01x02, J34 Conn_01x02, J35 Conn_01x02, J4 TERMBLOCK_1X2, J5 TERMBLOCK_1X2, J6 TERMBLOCK_1X2, J7 QWIIC_RIGHT_ANGLE, J7 TERMBLOCK_1X2, J8 TERMBLOCK_1X2, J9 TERMBLOCK_1X2, Q1 AOD417, U1 PCA9685, U10 LTV-817S, U11 LTV-817S, U12 LTV-817S, U13 LTV-817S, U14 LTV-817S, U15 LTV-817S, U2 DRV8870DDA, U2 K7805-2000R3L, U3 DRV8870DDA, U4 DRV8870DDA, U5 ADS1115IDGS, U6 ADS1115IDGS, U6 TCA9406DC, U7 MCP23008-xSO, U8 LTV-817S, U9 LTV-817S

Commit message: .
Parts:
- R29: value 1k -> 1k3
- R35: value 1k -> 270R
- R37, R38: value 1K -> 270R
- R4: value 1k -> 750R
Connections:
- net +5V: now also R37.1, R38.1
- net VCC: no longer R37.1, R38.1
Changed lines of the file:
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@@
   (junction (at 30.48 81.28) (diameter 0) (color 0 0 0 0)
   )
-  (junction (at 21.59 154.94) (diameter 0) (color 0 0 0 0)
-  )
-  (junction (at 21.59 149.86) (diameter 0) (color 0 0 0 0)
-  )
   (junction (at 280.67 158.75) (diameter 0) (color 0 0 0 0)
   )
@@
   (junction (at 63.5 81.28) (diameter 0) (color 0 0 0 0)
   )
+  (junction (at 21.59 154.94) (diameter 0) (color 0 0 0 0)
+  )
   (junction (at 384.81 46.99) (diameter 0) (color 0 0 0 0)
   )
@@
     (stroke (width 0.1524) (type solid))
   )
-  (wire (pts (xy 21.59 149.86) (xy 21.59 154.94))
-    (stroke (width 0) (type default))
-  )
   (wire (pts (xy 386.08 172.72) (xy 391.16 172.72))
     (stroke (width 0) (type default))
@@
       (effects (font (size 1.27 1.27)))
     )
-    (property "Value" "1k" (at 26.67 144.78 0)
+    (property "Value" "270R" (at 26.67 144.78 0)
       (effects (font (size 1.016 1.016) bold))
     )
@@
       (effects (font (size 1.27 1.27)))
     )
-    (property "Value" "1K" (at 26.67 154.94 0)
+    (property "Value" "270R" (at 26.67 154.94 0)
       (effects (font (size 1.016 1.016) bold))
     )
@@
     )
   )
+  (symbol (lib_id "power:+5V") (at 21.59 154.94 90) (unit 1)
+    (in_bom yes) (on_board yes) (dnp no) (fields_autoplaced)
+    (property "Reference" "#PWR069" (at 25.4 154.94 0)
+      (effects (font (size 1.27 1.27)) hide)
+    )
+    (property "Value" "+5V" (at 17.78 154.94 90)
+      (effects (font (size 1.27 1.27)) (justify left))
+    )
+    (property "Footprint" "" (at 21.59 154.94 0)
+      (effects (font (size 1.27 1.27)) hide)
+    )
+    (property "Datasheet" "" (at 21.59 154.94 0)
+      (effects (font (size 1.27 1.27)) hide)
+    )
+    (pin "1")
+    (instances
+      (project "Rev1"
+        (path "/89b827bc-676c-4335-87b0-d3946333fe72"
+          (reference "#PWR069") (unit 1)
+        )
+      )
+    )
+  )
   (symbol (lib_id "SparkFun ESP32 Thing Plus C-eagle-import:JUMPER-SMT_2_NC_TRACE_SILK") (at 196.85 151.13 90) (unit 1)
     (in_bom no) (on_board yes) (dnp no)
@@
       (effects (font (size 1.27 1.27)))
     )
-    (property "Value" "1k" (at 400.05 237.49 0)
+    (property "Value" "750R" (at 400.05 237.49 0)
       (effects (font (size 1.016 1.016) bold))
     )
@@
       (effects (font (size 1.27 1.27)))
     )
-    (property "Value" "1k" (at 359.41 44.45 0)
+    (property "Value" "1k3" (at 359.41 44.45 0)
       (effects (font (size 1.016 1.016) bold))
     )
@@
       (effects (font (size 1.27 1.27)))
     )
-    (property "Value" "1K" (at 26.67 160.02 0)
+    (property "Value" "270R" (at 26.67 160.02 0)
       (effects (font (size 1.016 1.016) bold))
     )
