File: Rev1/Rev1.kicad_sch (KiCad schematic)
At the start: 131 parts, among them J1 TERMBLOCK_1X2, J10 TERMBLOCK_1X2, J12 TERMBLOCK_1X2, J13 TERMBLOCK_1X2, J19 TERMBLOCK_1X2, J20 TERMBLOCK_1X2, J21 TERMBLOCK_1X2, J22 TERMBLOCK_1X2, J23 TERMBLOCK_1X2, J24 TERMBLOCK_1X2, J25 TERMBLOCK_1X2, J26 TERMBLOCK_1X2, J28 Conn_01x02, J29 Conn_01x02, J30 Conn_01x02, J31 Conn_01x02, J32 Conn_01x02, J33 Conn_01x02, J34 Conn_01x02, J35 Conn_01x02, J4 TERMBLOCK_1X2, J5 TERMBLOCK_1X2, J6 TERMBLOCK_1X2, J7 QWIIC_RIGHT_ANGLE, J7 TERMBLOCK_1X2, J8 TERMBLOCK_1X2, J9 TERMBLOCK_1X2, Q1 AOD417, U1 PCA9685, U10 LTV-817S, U11 LTV-817S, U12 LTV-817S, U13 LTV-817S, U14 LTV-817S, U15 LTV-817S, U2 DRV8870DDA, U3 DRV8870DDA, U3 K7805-2000R3L, U4 DRV8870DDA, U5 ADS1115IDGS, U6 ADS1115IDGS, U6 TCA9406DC, U7 MCP23008-xSO, U8 LTV-817S, U9 LTV-817S

Commit message: .
Connections:
- net +3.3V: now also JP3.5, JP4.5
- net SCL_A: now also JP3.3, JP4.3; no longer JP3.4, JP4.4
- net SDA_A: now also JP3.4, JP4.4; no longer JP3.3, JP4.3
- net OE: no longer names the net of R3.2, U1.23 (#OE)
- net OE: no longer JP3.5, JP4.5
Other:
- moved on the sheet: D2, J1, Q1, R3, R31

Commit message: .
Parts:
- removed J28, J29, J30, J31, J32, J33, J34, J35: Conn_01x02, Connector_PinHeader_2.54mm:PinHeader_1x02_P2.54mm_Vertical, symbol Connector_Generic:Conn_01x02
- removed JP3, JP4: PINHD-1X6CB, Adafruit PCA9685 rev C:1X06-CLEANBIG, symbol Adafruit PCA9685 rev C-eagle-import:PINHD-1X6CB
- added J3 (x2): Conn_01x05, Connector_PinHeader_2.54mm:PinHeader_1x05_P2.54mm_Vertical, symbol Connector_Generic:Conn_01x05
- A0, A1, A2, A3, A4, A5, JP5, LED1: now left out of the parts list
Connections:
- net +3.3V: now also J3.4 (Pin_4), J3.4 (Pin_4)
- net +5V: now also J3.1 (Pin_1), J3.1 (Pin_1)
- net GND: now also J3.5 (Pin_5), J3.5 (Pin_5); no longer J10.2, J12.2, J13.2
- net SCL_A: now also J3.2 (Pin_2), J3.2 (Pin_2)
- net SDA_A: now also J3.3 (Pin_3), J3.3 (Pin_3)
Other:
- moved on the sheet: C17, J19, J20, J21, J22, J23, J24, J25, J26, JP12, JP13, JP14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

Commit message: .
Parts:
- removed R15: 10K, Resistor_SMD:R_0603_1608Metric, symbol Adafruit PCA9685 rev C-eagle-import:RESISTOR0805_NOOUTLINE
- removed U7: MCP23008-xSO, Package_SO:SOIC-18W_7.5x11.6mm_P1.27mm, symbol Interface_Expansion:MCP23008-xSO
- added U7: TCA9534, PCM_Package_SO_AKL:TSSOP-16_4.4x5mm_P0.65mm, symbol Interface_Expansion:TCA9534
Connections:
- net +5V: now also U7.16 (VDD)
- net A0_1: now also U7.3 (A2)
- net A1_1: now also U7.2 (A1)
- net A2_1: now also U7.1 (A0)
- net GND: now also U7.8 (GND)
- net In0: now also U7.4 (P0)
- net In1: now also U7.5 (P1)
- net In2: now also U7.6 (P2)
- net In3: now also U7.7 (P3)
- net O0A: now also R22.1; no longer U12.4
- net O0B: now also U12.4; no longer R22.1
- net O1A: now also R24.1; no longer U13.4
- net O1B: now also U13.4; no longer R24.1
- net O2A: now also R26.1; no longer U14.4
- net O2B: now also U14.4; no longer R26.1
- net O3A: now also R28.1; no longer U15.4
- net O3B: now also U15.4; no longer R28.1
- net Out0: now also U7.9 (P4)
- net Out1: now also U7.10 (P5)
- net Out2: now also U7.11 (P6)
- net Out3: now also U7.12 (P7)
- net SCL_B: now also U7.14 (SCL)
- net SDA_B: now also U7.15 (SDA)
