File: Rev1/Rev1.kicad_pcb (KiCad board)
At the start: 2 copper layers, 67.3 x 96.9 mm, 143 parts, among them J1 TERMBLOCK_1X2, J10 TERMBLOCK_1X2, J12 TERMBLOCK_1X2, J13 TERMBLOCK_1X2, J19 TERMBLOCK_1X2, J2 QWIIC_RIGHT_ANGLE, J20 TERMBLOCK_1X2, J21 TERMBLOCK_1X2, J22 TERMBLOCK_1X2, J23 TERMBLOCK_1X2, J24 TERMBLOCK_1X2, J25 TERMBLOCK_1X2, J26 TERMBLOCK_1X2, J28 Conn_01x02, J29 Conn_01x02, J3 QWIIC_RIGHT_ANGLE, J30 Conn_01x02, J31 Conn_01x02, J32 Conn_01x02, J33 Conn_01x02, J34 Conn_01x02, J35 Conn_01x02, J4 TERMBLOCK_1X2, J5 TERMBLOCK_1X2, J6 TERMBLOCK_1X2, J7 TERMBLOCK_1X2, J8 TERMBLOCK_1X2, J9 TERMBLOCK_1X2, Q1 AOD417, U1 PCA9685, U10 PC817, U11 PC817, U12 PC817, U13 PC817, U14 PC817, U15 PC817, U16 ADS1115IDGS, U17 ADS1115IDGS, U2 DRV8870DDA, U3 DRV8870DDA, U4 DRV8870DDA, U5 K7805-2000R3L, U6 TCA9406DC, U7 MCP23008-xSO, U8 PC817, U9 PC817

Commit message: .
Parts:
- U10, U11, U12, U13, U14, U15, U8, U9: value PC817 -> LTV-817S; footprint Package_DIP:DIP-4_W7.62mm_SMDSocket_SmallPads -> PCM_Package_DIP_AKL:SMDIP-4_W9.53mm
- moved R8 31.5 mm to (140.4, 96.3), turned to 0 degrees
- moved R9 28.0 mm to (143.4, 96.3), turned to 0 degrees
- moved R17 25.8 mm to (146.4, 96.3), turned to 0 degrees
- moved R19 25.3 mm to (149.3, 96.3), turned to 0 degrees
- moved R26 22.9 mm to (123.1, 130.2), turned to 180 degrees
- moved R24 19.4 mm to (123.1, 120.7), turned to 180 degrees
- moved R28 18.8 mm to (123.1, 132.1), turned to 180 degrees
- moved R22 15.9 mm to (123.1, 111.1), turned to 180 degrees
- moved R23 13.2 mm to (138.2, 103.6), turned to -90 degrees
- moved R20 12.4 mm to (123.1, 101.5), turned to 180 degrees
- moved R25 12.3 mm to (138.2, 106.5), turned to -90 degrees
- moved R27 12.2 mm to (138.2, 109.5)
- moved R21 9.89 mm to (135.9, 92.5), turned to 0 degrees
- moved R18 9.03 mm to (123.1, 92.0), turned to 180 degrees
- moved G*** 5.93 mm to (133.9, 124.8)
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- renumbered R9 to R10, R10 to R9
Connections:
- U10 pad 1: Net-(R18-Pad1) -> /In3
- U10 pad 4: /In3 -> Net-(R18-Pad1)
- U11 pad 1: Net-(R20-Pad1) -> /In4
- U11 pad 4: /In4 -> Net-(R20-Pad1)
- U8 pad 1: Net-(R9-Pad1) -> /In1
- U8 pad 4: /In1 -> Net-(R9-Pad1)
- U9 pad 1: Net-(R16-Pad1) -> /In2
- U9 pad 4: /In2 -> Net-(R16-Pad1)
Routing:
- net +5V: track 649.6 -> 701.5 mm, vias 20 -> 13
- net Net-(R20-Pad1): track 2.80 -> 24.3 mm
- net Net-(R18-Pad1): track 2.69 -> 20.4 mm
- net /O4B: track 28.9 -> 11.4 mm
- net /Out2: track 17.5 -> 2.07 mm
- net /Out4: track 17.3 -> 3.24 mm
- net Net-(R16-Pad1): track 2.59 -> 16.5 mm
- net /In4: track 25.6 -> 38.2 mm
- net Net-(R23-Pad1): track 3.28 -> 15.0 mm
- net /Out3: track 14.1 -> 2.97 mm
- net Net-(R9-Pad1): track 2.51 -> 13.1 mm
- net Net-(R25-Pad1): track 2.56 -> 12.4 mm
- net /Out1: track 22.1 -> 12.4 mm
- net Net-(R27-Pad1): track 3.01 -> 12.2 mm
- net /In3: track 30.0 -> 39.1 mm
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
Commit message: .
Parts:
- R29: value 1k -> 1k3
- R35: value 1k -> 270R
- R37, R38: value 1K -> 270R
- R4: value 1k -> 750R
- moved C2 7.00 mm to (136.9, 136.2), turned to 90 degrees
- moved R37 4.74 mm to (154.7, 132.5), turned to -90 degrees
- moved U16 4.70 mm to (149.4, 132.2)
- moved C3 4.69 mm to (153.1, 132.5)
- moved R38 4.69 mm to (156.2, 132.5), turned to -90 degrees
- moved R35 3.51 mm to (150.6, 129.6), turned to 180 degrees
- moved G*** 2.36 mm to (145.1, 123.5)
- moved G*** 1.84 mm to (133.7, 126.6)
- moved U17 0.85 mm to (133.1, 136.5)
- moved R36 0.41 mm to (152.1, 127.3)
- moved R30 0.38 mm to (151.3, 125.1)
- moved J12 0.23 mm to (150.3, 137.6)
- moved J13 0.23 mm to (159.8, 137.6)
Connections:
- R37 pad 1: VCC -> +5V
- R38 pad 1: VCC -> +5V
Routing:
- net +5V: track 701.5 -> 747.1 mm, vias 13 -> 15
- net /Ain3: track 33.8 -> 15.9 mm
- net /Ain2: track 13.4 -> 29.2 mm
- net /SCL_B: track 152.4 -> 159.2 mm
- net VCC: track 295.6 -> 288.8 mm
- net /SDA_B: track 160.6 -> 166.8 mm
- net /Ain1: track 14.5 -> 9.82 mm
- net /Ain0: track 18.8 -> 14.4 mm
- net GND: track 114.1 -> 112.4 mm, vias 143 -> 141

Commit message: .
Parts:
- moved C2 1.06 mm to (136.9, 135.1)
- moved U17 1.06 mm to (133.1, 135.4)
Routing:
- net /Ain2: track 29.2 -> 12.1 mm
- net /Ain3: track 15.9 -> 25.2 mm
- net GND: track 112.4 -> 115.2 mm
- net /Ain7: track 3.51 -> 4.84 mm
- net /Ain6: track 2.81 -> 3.87 mm
- net /Ain5: track 2.31 -> 3.37 mm
- net /Ain4: track 4.00 -> 5.06 mm
- net +5V: track 747.1 -> 747.7 mm
Other:
- board text added: "1"
- board text added: "2"
- board text added: "3"
- board text added: "4"

Commit message: .
Parts:
- moved C18 1.68 mm to (164.4, 59.5)
- moved C19 1.68 mm to (156.4, 60.8)
- moved R32 1.68 mm to (156.4, 59.3)
- moved U6 1.68 mm to (160.8, 60.8)
Routing:
- net /SCL_B: track 158.8 -> 147.7 mm
- net +3.3V: track 92.0 -> 84.8 mm
- net +5V: track 747.7 -> 740.7 mm
- net /SDA_A: track 75.5 -> 69.2 mm
- net /SCL_A: track 71.1 -> 72.3 mm
- net GND: track 115.2 -> 114.9 mm, vias 141 -> 143
Other:
- board text added: "5"
- board text added: "6"
- board text added: "7"
- board text added: "8"

Commit message: .
Parts:
- removed JP11: JUMPER-SMT_2_NC_TRACE_SILK, OLIMEX_Jumpers-FP:SJ_Closed
- removed SJ_A0, SJ_A1, SJ_A2, SJ_A3, SJ_A4, SJ_A5: SOLDERJUMPERREFLOW_NOPASTE, Adafruit PCA9685 rev C:SOLDERJUMPER_REFLOW_NOPASTE
- removed TP1, TP2, TP3, TP4, TP5, TP6: TESTPOINTROUND1MM, Adafruit PCA9685 rev C:TESTPOINT_ROUND_1MM
- added A0: SolderJumper_2_Bridged, Jumper:SolderJumper-2_P1.3mm_Bridged_Pad1.0x1.5mm, F.Cu at (141.5, 52.1)
- added A1: SolderJumper_2_Bridged, Jumper:SolderJumper-2_P1.3mm_Bridged_Pad1.0x1.5mm, F.Cu at (139.0, 52.1)
- added A2: SolderJumper_2_Bridged, Jumper:SolderJumper-2_P1.3mm_Bridged_Pad1.0x1.5mm, F.Cu at (136.5, 52.1)
- added A3: SolderJumper_2_Bridged, Jumper:SolderJumper-2_P1.3mm_Bridged_Pad1.0x1.5mm, F.Cu at (133.9, 52.1)
- added A4: SolderJumper_2_Bridged, Jumper:SolderJumper-2_P1.3mm_Bridged_Pad1.0x1.5mm, F.Cu at (131.4, 52.1)
- added A5: SolderJumper_2_Bridged, Jumper:SolderJumper-2_P1.3mm_Bridged_Pad1.0x1.5mm, F.Cu at (128.8, 52.1)
- added JP10: SolderJumper_2_Bridged, Jumper:SolderJumper-2_P1.3mm_Bridged_Pad1.0x1.5mm, B.Cu at (149.7, 107.0)
- added JP6: SolderJumper_2_Bridged, Jumper:SolderJumper-2_P1.3mm_Bridged_Pad1.0x1.5mm, B.Cu at (155.2, 108.8)
- added LED0: SolderJumper_2_Bridged, Jumper:SolderJumper-2_P1.3mm_Bridged_Pad1.0x1.5mm, B.Cu at (121.9, 56.5)
- added LED1: SolderJumper_2_Bridged, Jumper:SolderJumper-2_P1.3mm_Bridged_Pad1.0x1.5mm, B.Cu at (122.0, 53.3)
- added R39: 10K, Resistor_SMD:R_0603_1608Metric, F.Cu at (144.2, 110.7)
- added R40: 10K, Resistor_SMD:R_0603_1608Metric, F.Cu at (145.7, 110.7)
- added R41: 10K, Resistor_SMD:R_0603_1608Metric, F.Cu at (147.2, 110.7)
- C1: value 10uF -> 0.1uF
- JP5, JP7, JP8, JP9: value JUMPER-SMT_2_NC_TRACE_SILK -> SolderJumper_2_Bridged; footprint OLIMEX_Jumpers-FP:SJ_Closed -> Jumper:SolderJumper-2_P1.3mm_Bridged_Pad1.0x1.5mm
- R21, R23, R25, R27: value 200R -> 380R
- R29: value 1k3 -> 2k2
- R4: value 750R -> 1k
- moved JP5 49.1 mm to (155.2, 89.7)
- moved JP7 38.3 mm to (155.2, 127.9), turned to 180 degrees
- moved JP9 24.1 mm to (149.7, 104.4)
- moved JP8 8.85 mm to (149.7, 101.9)
- moved C19 4.80 mm to (152.0, 62.8)
- moved U6 4.39 mm to (156.4, 60.8)
- moved C18 4.39 mm to (160.0, 59.5)
- moved R32 4.21 mm to (152.4, 60.5), turned to 90 degrees
- moved R34 3.75 mm to (142.7, 110.7), turned to 90 degrees
- moved J31 2.55 mm to (123.5, 96.4), turned to 0 degrees
- moved J32 2.55 mm to (123.5, 106.0), turned to 0 degrees
- moved J35 2.55 mm to (123.5, 134.6), turned to 0 degrees
- moved J28 2.55 mm to (123.5, 67.7), turned to 0 degrees
- moved J29 2.55 mm to (123.5, 77.3), turned to 0 degrees
- moved J30 2.55 mm to (123.5, 86.8), turned to 0 degrees
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Connections:
- J19 pad 2: /I1 -> /I0
- J20 pad 2: /I2 -> /I1
- J21 pad 2: /I3 -> /I2
- J22 pad 2: /I4 -> /I3
- J23 pad 1: /O1A -> /O0A
- J23 pad 2: /O1B -> /O0B
- J24 pad 1: /O2A -> /O1A
- J24 pad 2: /O2B -> /O1B
- J25 pad 1: /O3A -> /O2A
- J25 pad 2: /O3B -> /O2B
- J26 pad 1: /O4A -> /O3A
- J26 pad 2: /O4B -> /O3B
- J28 pad 1: /I1 -> +5V
- J28 pad 2: +5V -> /I0
- J29 pad 1: /I2 -> +5V
- J29 pad 2: +5V -> /I1
- J30 pad 1: /I3 -> +5V
- J30 pad 2: +5V -> /I2
- J31 pad 1: /I4 -> +5V
- J31 pad 2: +5V -> /I3
- J32 pad 1: /O1B -> /O0A
- J32 pad 2: /O1A -> /O0B
- J33 pad 1: /O2B -> /O1A
- J33 pad 2: /O2A -> /O1B
- J34 pad 1: /O3B -> /O2A
- J34 pad 2: /O3A -> /O2B
- J35 pad 1: /O4B -> /O3A
- J35 pad 2: /O4A -> /O3B
- JP5 pad 1: Net-(D3-A) -> +5V
- JP5 pad 2: +3.3V -> Net-(JP5-B)
- JP7 pad 1: Net-(U2-VREF) -> +5V
- JP7 pad 2: +5V -> Net-(JP7-B)
- JP8 pad 1: Net-(U3-VREF) -> /A0_1
- JP8 pad 2: +5V -> GND
- JP9 pad 1: Net-(U4-VREF) -> /A1_1
- JP9 pad 2: +5V -> GND
- R1 pad 1: GND -> +5V
- R1 pad 2: GND -> +5V
- R1 pad 3: GND -> +5V
- R1 pad 4: GND -> +5V
- R10 pad 2: /I1 -> /I0
- R16 pad 2: /I2 -> /I1
- R17 pad 1: /In3 -> /In2
- R18 pad 2: /I3 -> /I2
- R19 pad 1: /In4 -> /In3
- R2 pad 1: GND -> +5V
- R2 pad 2: GND -> +5V
- R20 pad 2: /I4 -> /I3
- R21 pad 2: /Out1 -> /Out0
- R22 pad 1: /O1B -> /O0B
- R23 pad 2: /Out2 -> /Out1
- R24 pad 1: /O2B -> /O1B
- R25 pad 2: /Out3 -> /Out2
- R26 pad 1: /O3B -> /O2B
- R27 pad 2: /Out4 -> /Out3
- R28 pad 1: /O4B -> /O3B
- R29 pad 1: GND -> Net-(D1-K)
- R29 pad 2: Net-(D1-K) -> GND
- R32 pad 1: +3.3V -> +5V
- R32 pad 2: GND -> Net-(U6-OE)
- R4 pad 1: GND -> Net-(D3-K)
- R4 pad 2: Net-(D3-K) -> GND
- R8 pad 1: /In1 -> /In0
- R9 pad 1: /In2 -> /In1
- U10 pad 1: /In3 -> Net-(R18-Pad1)
- U10 pad 4: Net-(R18-Pad1) -> /In2
- U11 pad 1: /In4 -> Net-(R20-Pad1)
- U11 pad 4: Net-(R20-Pad1) -> /In3
- U12 pad 4: /O1A -> /O0A
- U13 pad 4: /O2A -> /O1A
- U14 pad 4: /O3A -> /O2A
- U15 pad 4: /O4A -> /O3A
- U2 pad 4: Net-(U2-VREF) -> Net-(JP5-B)
- U3 pad 4: Net-(U3-VREF) -> Net-(JP6-B)
- U4 pad 4: Net-(U4-VREF) -> Net-(JP7-B)
- U6 pad 6: +3.3V -> Net-(U6-OE)
- U7 pad 10: /In1 -> /In0
- U7 pad 11: /In2 -> /In1
- U7 pad 12: /In3 -> /In2
- U7 pad 13: /In4 -> /In3
- U7 pad 14: /Out1 -> /Out0
- U7 pad 15: /Out2 -> /Out1
- U7 pad 16: /Out3 -> /Out2
- U7 pad 17: /Out4 -> /Out3
- U7 pad 3: GND -> /A2_1
- U7 pad 4: GND -> /A1_1
- U7 pad 5: GND -> /A0_1
- U8 pad 1: /In1 -> Net-(R10-Pad1)
- U8 pad 4: Net-(R10-Pad1) -> /In0
- U9 pad 1: /In2 -> Net-(R16-Pad1)
- U9 pad 4: Net-(R16-Pad1) -> /In1
Routing:
- net /In4: track 38.2 -> 0.00 mm
- net /O4A: track 34.0 -> 0.00 mm
- net /In0: track 0.00 -> 29.1 mm
- net /O0A: track 0.00 -> 25.4 mm
- net /O0B: track 0.00 -> 17.9 mm
- net GND: track 114.9 -> 128.8 mm, vias 143 -> 149
- net /In2: track 40.9 -> 27.2 mm
- net /I4: track 13.3 -> 0.00 mm
- net /I0: track 0.00 -> 13.3 mm
- net +5V: track 740.7 -> 753.4 mm
- net /In3: track 39.1 -> 26.7 mm
- net /Out0: track 0.00 -> 12.4 mm
- net /SDA_B: track 166.0 -> 154.0 mm
- net /In1: track 40.9 -> 29.1 mm
- net /O4B: track 11.4 -> 0.00 mm
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Other:
- board text removed: "A0"
- board text removed: "A1"
- board text removed: "A2"
- board text removed: "A3"
- board text removed: "A4"
- board text removed: "A5"

Commit message: .
Parts:
- A0, A1, A2, A3, A4, A5: moved to B.Cu
Connections:
- JP3 pad 3: /SDA_A -> /SCL_A
- JP3 pad 4: /SCL_A -> /SDA_A
- JP3 pad 5: /OE -> +3.3V
- JP4 pad 3: /SDA_A -> /SCL_A
- JP4 pad 4: /SCL_A -> /SDA_A
- JP4 pad 5: /OE -> +3.3V
- R3 pad 2: /OE -> Net-(U1-#OE)
- U1 pad 23: /OE -> Net-(U1-#OE)
Routing:
- net /OE: track 58.5 -> 0.00 mm, vias 3 -> 0
- net +3.3V: track 79.9 -> 114.7 mm, vias 4 -> 3
- net Net-(U1-#OE): track 0.00 -> 11.2 mm, vias 0 -> 2
- net /SCL_A: track 78.2 -> 86.1 mm, vias 3 -> 5
- net GND: track 128.8 -> 131.7 mm, vias 149 -> 146
- net /SDA_A: track 66.0 -> 66.9 mm
- net /A2: track 16.9 -> 16.3 mm
