File: Rev1/Rev1.kicad_pcb (KiCad board)
At the start: 2 copper layers, 67.3 x 96.9 mm, 143 parts, among them J1 TERMBLOCK_1X2, J10 TERMBLOCK_1X2, J12 TERMBLOCK_1X2, J13 TERMBLOCK_1X2, J19 TERMBLOCK_1X2, J2 QWIIC_RIGHT_ANGLE, J20 TERMBLOCK_1X2, J21 TERMBLOCK_1X2, J22 TERMBLOCK_1X2, J23 TERMBLOCK_1X2, J24 TERMBLOCK_1X2, J25 TERMBLOCK_1X2, J26 TERMBLOCK_1X2, J28 Conn_01x02, J29 Conn_01x02, J3 QWIIC_RIGHT_ANGLE, J30 Conn_01x02, J31 Conn_01x02, J32 Conn_01x02, J33 Conn_01x02, J34 Conn_01x02, J35 Conn_01x02, J4 TERMBLOCK_1X2, J5 TERMBLOCK_1X2, J6 TERMBLOCK_1X2, J7 TERMBLOCK_1X2, J8 TERMBLOCK_1X2, J9 TERMBLOCK_1X2, Q1 AOD417, U1 PCA9685, U10 LTV-817S, U11 LTV-817S, U12 LTV-817S, U13 LTV-817S, U14 LTV-817S, U15 LTV-817S, U16 ADS1115IDGS, U17 ADS1115IDGS, U2 DRV8870DDA, U3 DRV8870DDA, U4 DRV8870DDA, U5 K7805-2000R3L, U6 TCA9406DC, U7 MCP23008-xSO, U8 LTV-817S, U9 LTV-817S

Commit message: .
Parts:
- added Sign-RecyclBin: , OLIMEX_LOGOs-FP:LOGO_RECYCLEBIN_1, B.Cu at (157.6, 68.5)
- moved G*** 2.43 mm to (144.5, 110.5)
- moved Sign_Pb-Free 1.69 mm to (160.3, 65.3)

Commit message: .
Parts:
- removed J28, J29, J30, J31, J32, J33, J34, J35: Conn_01x02, Connector_PinHeader_2.54mm:PinHeader_1x02_P2.54mm_Vertical
- removed JP3, JP4: PINHD-1X6CB, Adafruit PCA9685 rev C:1X06-CLEANBIG
- added ?: STAND-OFF, Qwiic_BME688:STAND-OFF, F.Cu at (104.6, 53.6)
- added J11: Conn_01x05, Connector_PinHeader_2.54mm:PinHeader_1x05_P2.54mm_Vertical, F.Cu at (119.0, 61.3)
- added J14: Conn_01x05, Connector_PinHeader_2.54mm:PinHeader_1x05_P2.54mm_Vertical, F.Cu at (167.7, 61.3)
- moved Sign_Pb-Free 6.86 mm to (153.5, 65.3)
- moved Sign-RecyclBin 4.11 mm to (161.7, 68.6)
- moved G*** 3.59 mm to (143.0, 126.4)
- moved G*** 1.34 mm to (132.4, 126.4) (x2)
- moved R30 0.37 mm to (151.3, 124.7)
- moved R36 0.37 mm to (152.1, 127.0)
Connections:
- J10 pad 2: GND -> unconnected-(J10-Pad2)
- J12 pad 2: GND -> unconnected-(J12-Pad2)
- J13 pad 2: GND -> unconnected-(J13-Pad2)
Routing:
- net VCC: track 291.8 -> 201.7 mm
- net +5V: track 753.1 -> 685.1 mm
- net /O0B: track 17.9 -> 6.58 mm
- net /O2B: track 18.2 -> 6.93 mm
- net /O1B: track 17.3 -> 6.58 mm
- net /I2: track 14.3 -> 4.88 mm
- net /I1: track 13.3 -> 4.89 mm
- net /I0: track 13.3 -> 4.88 mm
- net /I3: track 13.3 -> 4.88 mm
- net /O3B: track 11.4 -> 8.28 mm
- net /O2A: track 33.2 -> 31.2 mm
- net /O1A: track 29.3 -> 27.3 mm
- net /O0A: track 25.4 -> 23.4 mm
- net /O3A: track 34.0 -> 32.2 mm
- net /SCL_A: track 86.1 -> 84.7 mm
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Other:
- board text added: "+3V"
- board text added: "+5V"
- board text added: "Rev.1"
- board text removed: "5V+"
- board text removed: "I2C->"
- board text removed: "OE"
- board text removed: "VCC"

Commit message: .
Parts:
- removed ?: STAND-OFF, Qwiic_BME688:STAND-OFF
- removed R15: 10K, Resistor_SMD:R_0603_1608Metric
- U7: value MCP23008-xSO -> TCA9534; footprint Package_SO:SOIC-18W_7.5x11.6mm_P1.27mm -> PCM_Package_SO_AKL:TSSOP-16_4.4x5mm_P0.65mm
- moved C12 26.7 mm to (133.1, 64.2), turned to 90 degrees
- moved G*** 15.8 mm to (148.1, 60.4)
- moved R20 15.7 mm to (124.5, 85.9), turned to -90 degrees
- moved C17 15.4 mm to (146.9, 97.1), turned to 90 degrees
- moved R23 15.1 mm to (124.5, 97.2)
- moved R34 14.2 mm to (150.3, 98.7), turned to -90 degrees
- moved R25 14.1 mm to (124.5, 102.8)
- moved R27 13.7 mm to (124.5, 108.5), turned to -90 degrees
- moved JP10 13.1 mm to (140.8, 97.3), turned to 180 degrees
- moved R33 12.0 mm to (148.8, 98.7), turned to -90 degrees
- moved R18 11.8 mm to (124.5, 80.3), turned to -90 degrees
- moved R21 11.4 mm to (124.5, 91.5), turned to -90 degrees
- moved C1 10.5 mm to (135.7, 56.2)
- moved JP9 9.96 mm to (140.8, 99.9), turned to 180 degrees
- moved R41 9.58 mm to (150.6, 101.7), turned to 0 degrees
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Connections:
- R22 pad 1: /O0B -> /O0A
- R24 pad 1: /O1B -> /O1A
- R26 pad 1: /O2B -> /O2A
- R28 pad 1: /O3B -> /O3A
- U12 pad 4: /O0A -> /O0B
- U13 pad 4: /O1A -> /O1B
- U14 pad 4: /O2A -> /O2B
- U15 pad 4: /O3A -> /O3B
- U7 pad 1: /SCL_B -> /A2_1
- U7 pad 10: /In0 -> /Out1
- U7 pad 11: /In1 -> /Out2
- U7 pad 12: /In2 -> /Out3
- U7 pad 13: /In3 -> unconnected-(U7-~{INT}-Pad13)
- U7 pad 14: /Out0 -> /SCL_B
- U7 pad 15: /Out1 -> /SDA_B
- U7 pad 16: /Out2 -> +5V
- U7 pad 2: /SDA_B -> /A1_1
- U7 pad 3: /A2_1 -> /A0_1
- U7 pad 4: /A1_1 -> /In0
- U7 pad 5: /A0_1 -> /In1
- U7 pad 6: Net-(U7-~{RESET}) -> /In2
- U7 pad 7: unconnected-(U7-NC-Pad7) -> /In3
- U7 pad 8: unconnected-(U7-INT-Pad8) -> GND
- U7 pad 9: GND -> /Out0
Routing:
- net GND: track 130.8 -> 45.4 mm, vias 146 -> 118
- net +5V: track 685.1 -> 607.6 mm, vias 15 -> 14
- net /Out3: track 3.24 -> 32.6 mm
- net /O3B: track 8.28 -> 36.6 mm, vias 0 -> 1
- net /Out1: track 2.07 -> 29.5 mm
- net /O3A: track 32.2 -> 6.15 mm
- net /O2B: track 6.93 -> 32.7 mm, vias 0 -> 1
- net /O2A: track 31.2 -> 6.14 mm
- net /Out2: track 2.97 -> 27.8 mm
- net /O1B: track 6.58 -> 28.8 mm, vias 0 -> 1
- net /O1A: track 27.3 -> 6.14 mm
- net /Out0: track 12.4 -> 32.3 mm
- net /O0B: track 6.58 -> 25.1 mm, vias 0 -> 1
- net /O0A: track 23.4 -> 6.14 mm
- net /P12: track 6.16 -> 20.9 mm
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